File: hw/KeyboardPCB/_autosave-KeyboardPCB.kicad_pcb (KiCad board)
At the start: 2 copper layers, 335 x 100 mm, 164 parts, among them IC1 TPS2113ADRBR, IC2 BGM220PC22HNA2R, J1 USB_B_Micro, J2 Conn_01x07_Pin, J3 Conn_01x06_Pin, J4 Conn_02x05_Odd_Even, J5 BATT_POS, J6 BATT_NEG, K1 KEYSW, K10 KEYSW, K11 KEYSW, K12 KEYSW, K13 KEYSW, K14 KEYSW, K15 KEYSW, K16 KEYSW, K17 KEYSW, K18 KEYSW, K19 KEYSW, K2 KEYSW, K20 KEYSW, K21 KEYSW, K22 KEYSW, K23 KEYSW, K24 KEYSW, K25 KEYSW, K26 KEYSW, K27 KEYSW, K28 KEYSW, K29 KEYSW, K3 KEYSW, K30 KEYSW, K31 KEYSW, K32 KEYSW, K33 KEYSW, K34 KEYSW, K35 KEYSW, K36 KEYSW, K37 KEYSW, K38 KEYSW, K39 KEYSW, K4 KEYSW, K40 KEYSW, K41 KEYSW, K42 KEYSW, K43 KEYSW, K44 KEYSW, K45 KEYSW, K46 KEYSW, K47 KEYSW, K48 KEYSW, K49 KEYSW, K5 KEYSW, K50 KEYSW, K51 KEYSW, K52 KEYSW, K53 KEYSW, K54 KEYSW, K55 KEYSW, K56 KEYSW, K57 KEYSW, K58 KEYSW, K59 KEYSW, K6 KEYSW, K60 KEYSW, K61 KEYSW, K62 KEYSW, K7 KEYSW, K8 KEYSW, K9 KEYSW, SW2 BAT_SWITCH, U1 TM4C123GH6PMI7, U2 TPS73633DBV, U3 Adafruit ST7735R, X2 16MHz

Commit message: Lotta Changes, Initial Routing
Parts:
- added REF**: RGB-6028, Keebio-Parts.pretty-master:RGB-6028, F.Cu at (644.0, 151.3)
- added REF**: RGB_BRAG, Keebio-Parts.pretty-master:RGB_3528_Blue_Notch, F.Cu at (653.0, 158.2)
Changed lines of the file:
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@@
     )
+  )
+  (footprint "Keebio-Parts.pretty-master:RGB-6028" (layer "F.Cu")
+    (at 643.95 151.3)
+    (attr smd)
+    (fp_text reference "REF**" (at 0 8) (layer "F.SilkS")
+        (effects (font (size 1 1) (thickness 0.15)))
+    )
+    (fp_text value "RGB-6028" (at 0 2.3) (layer "F.Fab")
+        (effects (font (size 1 1) (thickness 0.15)))
+    )
+    (fp_circle (center -2.5 6.8) (end -2.5 6.6)
+      (stroke (width 0.15) (type solid)) (fill none) (layer "F.SilkS"))
+    (fp_line (start -9.525 -9.525) (end 9.525 -9.525)
+      (stroke (width 0.15) (type solid)) (layer "Dwgs.User"))
+    (fp_line (start -9.525 9.525) (end -9.525 -9.525)
+      (stroke (width 0.15) (type solid)) (layer "Dwgs.User"))
+    (fp_line (start 9.525 -9.525) (end 9.525 9.525)
+      (stroke (width 0.15) (type solid)) (layer "Dwgs.User"))
+    (fp_line (start 9.525 9.525) (end -9.525 9.525)
+      (stroke (width 0.15) (type solid)) (layer "Dwgs.User"))
+    (fp_line (start -1.9 3.38) (end -1.9 6.78)
+      (stroke (width 0.15) (type solid)) (layer "Edge.Cuts"))
+    (fp_line (start 1.9 3.38) (end -1.9 3.38)
+      (stroke (width 0.15) (type solid)) (layer "Edge.Cuts"))
+    (fp_line (start 1.9 3.38) (end 1.9 6.78)
+      (stroke (width 0.15) (type solid)) (layer "Edge.Cuts"))
+    (fp_line (start 1.9 6.78) (end -1.9 6.78)
+      (stroke (width 0.15) (type solid)) (layer "Edge.Cuts"))
+    (pad "1" smd rect (at -2.595 4.33) (size 1.19 0.9) (layers "F.Cu" "F.Paste" "F.Mask"))
+    (pad "2" smd rect (at 2.595 5.83) (size 1.19 0.9) (layers "F.Cu" "F.Paste" "F.Mask"))
+    (pad "3" smd rect (at 2.595 4.33) (size 1.19 0.9) (layers "F.Cu" "F.Paste" "F.Mask"))
+    (pad "4" smd rect (at -2.595 5.83) (size 1.19 0.9) (layers "F.Cu" "F.Paste" "F.Mask"))
   )
   (footprint "MX_Hotswap:MX-Hotswap-1U" (layer "F.Cu")
@@
       (net 32 "Net-(D19-K)") (pintype "passive"))
   )
+  (footprint "Keebio-Parts.pretty-master:RGB_3528_Blue_Notch" (layer "F.Cu")
+    (at 653 158.2)
+    (descr "RGB LED 3.2x2.7mm http://www.avagotech.com/docs/AV02-0610EN")
+    (tags "LED 3227")
+    (attr smd)
+    (fp_text reference "REF**" (at 0 2.5) (layer "F.SilkS")
+        (effects (font (size 0.7 0.7) (thickness 0.15)))
+    )
+    (fp_text value "RGB_BRAG" (at 0 -2.5) (layer "F.Fab")
+        (effects (font (size 0.7 0.7) (thickness 0.15)))
+    )
+    (fp_text user "R" (at -4.2 -0.75) (layer "F.SilkS")
+        (effects (font (size 0.7 0.7) (thickness 0.15)))
+    )
+    (fp_text user "G" (at -4.2 0.75) (layer "F.SilkS")
+        (effects (font (size 0.7 0.7) (thickness 0.15)))
+    )
+    (fp_text user "+" (at 4.2 0.75) (layer "F.SilkS")
+        (effects (font (size 0.7 0.7) (thickness 0.15)))
+    )
+    (fp_text user "B" (at 4.2 -0.75) (layer "F.SilkS")
+        (effects (font (size 0.7 0.7) (thickness 0.15)))
+    )
+    (fp_line (start -2 -1.8) (end 2 -1.8)
+      (stroke (width 0.15) (type solid)) (layer "F.SilkS"))
+    (fp_line (start -2 1.8) (end -2 -1.8)
+      (stroke (width 0.15) (type solid)) (layer "F.SilkS"))
+    (fp_line (start 2 -1.8) (end 2 1.8)
+      (stroke (width 0.15) (type solid)) (layer "F.SilkS"))
+    (fp_line (start 2 1.8) (end -2 1.8)
+      (stroke (width 0.15) (type solid)) (layer "F.SilkS"))
+    (fp_circle (center 2.5 -1.5) (end 2.6 -1.3)
+      (stroke (width 0.15) (type solid)) (fill none) (layer "F.SilkS"))
+    (fp_line (start -1.6 -1.4) (end -1.6 1.4)
+      (stroke (width 0.12) (type solid)) (layer "Cmts.User"))
+    (fp_line (start -1.6 1.4) (end 1.6 1.4)
+      (stroke (width 0.12) (type solid)) (layer "Cmts.User"))
+    (fp_line (start 0.7 1.4) (end 0.7 -1.4)
+      (stroke (width 0.12) (type solid)) (layer "Cmts.User"))
+    (fp_line (start 1.2 -1.4) (end -1.6 -1.4)
+      (stroke (width 0.12) (type solid)) (layer "Cmts.User"))
+    (fp_line (start 1.2 -1.4) (end 1.2 1.4)
+      (stroke (width 0.12) (type solid)) (layer "Cmts.User"))
+    (fp_line (start 1.6 -1) (end 1.2 -1.4)
+      (stroke (width 0.12) (type solid)) (layer "Cmts.User"))
+    (fp_line (start 1.6 1.4) (end 1.6 -1)
+      (stroke (width 0.12) (type solid)) (layer "Cmts.User"))
+    (fp_line (start -1.8 -1.6) (end 1.8 -1.6)
+      (stroke (width 0.15) (type solid)) (layer "Edge.Cuts"))
+    (fp_line (start -1.8 1.6) (end -1.8 -1.6)
+      (stroke (width 0.15) (type solid)) (layer "Edge.Cuts"))
+    (fp_line (start -1.8 1.6) (end 1.8 1.6)
+      (stroke (width 0.15) (type solid)) (layer "Edge.Cuts"))
+    (fp_line (start 1.8 1.6) (end 1.8 -1.6)
+      (stroke (width 0.15) (type solid)) (layer "Edge.Cuts"))
+    (fp_line (start -3.7 -1.65) (end 3.7 -1.65)
+      (stroke (width 0.05) (type solid)) (layer "B.CrtYd"))
+    (fp_line (start -3.7 1.65) (end -3.7 -1.65)
+      (stroke (width 0.05) (type solid)) (layer "B.CrtYd"))
+    (fp_line (start 3.7 -1.65) (end 3.7 1.65)
+      (stroke (width 0.05) (type solid)) (layer "B.CrtYd"))
+    (fp_line (start 3.7 1.65) (end -3.7 1.65)
+      (stroke (width 0.05) (type solid)) (layer "B.CrtYd"))
+    (pad "1" smd rect (at 2.6 -0.75) (size 2 0.7) (layers "F.Cu" "F.Paste" "F.Mask"))
+    (pad "2" smd rect (at -2.6 -0.75) (size 2 0.7) (layers "F.Cu" "F.Paste" "F.Mask"))
+    (pad "3" smd rect (at 2.6 0.75) (size 2 0.7) (layers "F.Cu" "F.Paste" "F.Mask"))
+    (pad "4" smd rect (at -2.6 0.75) (size 2 0.7) (layers "F.Cu" "F.Paste" "F.Mask"))
+  )
   (footprint "footprints:adafruit_st7735r" (layer "F.Cu")
