File: hw/PCB/PCB.kicad_sch (KiCad schematic)
At the start: 331 parts, among them IC2 BGM220PC22HNA2R, J1 USB_C_Receptacle_USB2.0, J2 Conn_ARM_JTAG_SWD_10, J4 USB_B_Micro, J7 ${ALTIUM_VALUE}, K1 KEYSW, K10 KEYSW, K100 KEYSW, K101 KEYSW, K102 KEYSW, K103 KEYSW, K104 KEYSW, K105 KEYSW, K106 KEYSW, K107 KEYSW, K108 KEYSW, K109 KEYSW, K11 KEYSW, K110 KEYSW, K111 KEYSW, K112 KEYSW, K113 KEYSW, K114 KEYSW, K115 KEYSW, K116 KEYSW, K117 KEYSW, K118 KEYSW, K119 KEYSW, K12 KEYSW, K120 KEYSW, K121 KEYSW, K122 KEYSW, K123 KEYSW, K124 KEYSW, K13 KEYSW, K14 KEYSW, K15 KEYSW, K16 KEYSW, K17 KEYSW, K18 KEYSW, K19 KEYSW, K2 KEYSW, K20 KEYSW, K21 KEYSW, K22 KEYSW, K23 KEYSW, K24 KEYSW, K25 KEYSW, K26 KEYSW, K27 KEYSW, K28 KEYSW, K29 KEYSW, K3 KEYSW, K30 KEYSW, K31 KEYSW, K32 KEYSW, K33 KEYSW, K34 KEYSW, K35 KEYSW, K36 KEYSW, K37 KEYSW, K38 KEYSW, K39 KEYSW, K4 KEYSW, K40 KEYSW, K41 KEYSW, K42 KEYSW, K43 KEYSW, K44 KEYSW, K45 KEYSW, K46 KEYSW, K47 KEYSW, K48 KEYSW, K49 KEYSW, K5 KEYSW, K50 KEYSW, K51 KEYSW, K52 KEYSW, K53 KEYSW, K54 KEYSW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

Commit message: Slight tweak to keyboard matrix
Parts:
- removed D10, D108, D11, D110, D12, D121, D13, D14, D15, D16, D17, D18, D19, D20, D21, D22, D23, D24, D25, D26, D27, D28, D29, D30, D31, D32, D33, D34, D35, D36, D37, D38, D39, D40, D41, D42, D43, D44, D45, D46, D47, D48, D49, D50, D51, D52, D53, D54, D55, D56, D57, D58, D59, D60, D61, D62, D63, D64, D65: D, Diode_SMD:D_SOD-123, symbol Device:D
- removed K1, K10, K11, K12, K13, K15, K16, K17, K18, K19, K20, K21, K22, K23, K24, K25, K26, K28, K29, K30, K31, K32, K33, K34, K35, K36, K37, K38, K39, K40, K41, K42, K43, K45, K46, K47, K48, K50, K51, K52, K53, K55, K56, K8: KEYSW, MX_Hotswap:MX-Hotswap-1U, symbol keyboard_parts:KEYSW
- removed K106, K14, K44, K49, K54, K58, K62, K9: KEYSW, MX_Hotswap:MX-Hotswap-1.25U, symbol keyboard_parts:KEYSW
- removed K119, K57, K60: KEYSW, MX_Hotswap:MX-Hotswap-1.5U, symbol keyboard_parts:KEYSW
- removed K121, K59: KEYSW, MX_Hotswap:MX-Hotswap-2U, symbol keyboard_parts:KEYSW
- removed K27: KEYSW, MX_Hotswap:MX-Hotswap-6.25U, symbol keyboard_parts:KEYSW
- removed K61: KEYSW, MX_Hotswap:MX-Hotswap-2.25U, symbol keyboard_parts:KEYSW
- added D127, D128, D129, D130, D131, D132, D133, D134, D135, D136, D137, D138, D139, D140, D141, D142, D143, D144, D145, D146, D147, D148, D149, D150, D151, D152, D153, D154, D155, D156, D157, D158, D159, D160, D161, D162, D163, D164, D165, D166, D167, D168, D169, D170, D171, D172, D173, D174, D175, D176, D177, D178, D179, D180, D181, D182, D183, D184, D185, D186, D187, D188, D189, D190, D191, D192, D193, D194, D195, D196: WS2812B, LED_SMD:LED_WS2812B_PLCC4_5.0x5.0mm_P3.2mm, symbol LED:WS2812B
- K2: footprint MX_Hotswap:MX-Hotswap-1.5U -> MX_Hotswap:MX-Hotswap-1.25U
- K3: footprint MX_Hotswap:MX-Hotswap-1.75U -> MX_Hotswap:MX-Hotswap-1.5U
- K5: footprint MX_Hotswap:MX-Hotswap-1.25U -> MX_Hotswap:MX-Hotswap-2.25U
- K6, K7: footprint MX_Hotswap:MX-Hotswap-1U -> MX_Hotswap:MX-Hotswap-2.25U
- renumbered K63 to K01
Connections:
- net JTAG_SWO_TDO: now also D4.2 (A), D9.2 (A); no longer D8.2 (A)
- net col0: no longer K2.1, K3.1, K4.1, K5.1
- net col1: now also K4.1; no longer K6.1, K7.1
- net col10: no longer K107.1, K108.1, K109.1, K110.1, K111.1
- net col12: now also K5.1, K6.1
- net col13: now also K2.1, K3.1
- net col9: now also K7.1
- net row0: no longer D4.2 (A), D9.2 (A)
- net row2: now also D7.2 (A); no longer D6.2 (A)
- net row3: now also D6.2 (A), D8.2 (A); no longer D7.2 (A)
- net at D7.1 (K): now also K5.2; no longer K4.2
- net at K108.2: now also D5.1 (K)
- net at D4.1 (K): now also K2.2
- net at D8.1 (K): now also K6.2; no longer K5.2
- net at D123.1 (K): now also K3.2
- net at D6.1 (K): now also K4.2; no longer K3.2
- net at K7.2: now also D9.1 (K)
- new net: K107.1, K108.1, K109.1, K110.1, K111.1

Commit message: LEDs!
Parts:
- removed D128, D129, D130, D131, D133, D134, D135, D136, D138, D139, D140, D141, D143, D144, D145, D146, D148, D149, D150, D151, D153, D154, D155, D156, D158, D159, D160, D161, D163, D164, D165, D166, D168, D169, D170, D171, D173, D174, D175, D176, D178, D179, D180, D181, D183, D184, D185, D186, D188, D189, D190, D191, D192, D193, D194, D195, D196: WS2812B, LED_SMD:LED_WS2812B_PLCC4_5.0x5.0mm_P3.2mm, symbol LED:WS2812B
- removed X2: ${ALTIUM_VALUE}, XTAL_2012, symbol nrf5340_qkaa_config2-altium-import:root_3_XTAL_2-pin
- added D10, D108, D11, D12, D13, D14, D15, D16, D17, D18, D19, D20, D21, D22, D23, D24, D25, D26, D27, D28, D29, D30, D31, D32, D33, D34, D35, D36, D37, D38, D39, D40, D41, D42, D43, D44, D45, D46, D47, D48, D49, D50, D51, D52, D53, D54, D55, D58, D62, D63, D64, D65: WS2812B, LED_SMD:LED_WS2812B_PLCC4_5.0x5.0mm_P3.2mm, symbol LED:WS2812B
Connections:
- net P0.00/XL1 is gone; now on net ROW0_LED: U4.N1 (P0.00/XL1)
- net GND: now also D127.3 (VSS), D132.3 (VSS), D137.3 (VSS), D142.3 (VSS), D147.3 (VSS), D152.3 (VSS), D157.3 (VSS), D162.3 (VSS), D167.3 (VSS), D172.3 (VSS), D177.3 (VSS), D182.3 (VSS), D187.3 (VSS), D10.3 (VSS), D108.3 (VSS), D11.3 (VSS), D12.3 (VSS), D13.3 (VSS), D14.3 (VSS), D15.3 (VSS), D16.3 (VSS), D17.3 (VSS), D18.3 (VSS), D19.3 (VSS), D20.3 (VSS), D21.3 (VSS), D22.3 (VSS), D23.3 (VSS), D24.3 (VSS), D25.3 (VSS), D26.3 (VSS), D27.3 (VSS), D28.3 (VSS), D29.3 (VSS), D30.3 (VSS), D31.3 (VSS), D32.3 (VSS), D33.3 (VSS), D34.3 (VSS), D35.3 (VSS), D36.3 (VSS), D37.3 (VSS), D38.3 (VSS), D39.3 (VSS), D40.3 (VSS), D41.3 (VSS), D42.3 (VSS), D43.3 (VSS), D44.3 (VSS), D45.3 (VSS), D46.3 (VSS), D47.3 (VSS), D48.3 (VSS), D49.3 (VSS), D50.3 (VSS), D51.3 (VSS), D52.3 (VSS), D53.3 (VSS), D54.3 (VSS), D55.3 (VSS), D58.3 (VSS), D62.3 (VSS), D63.3 (VSS), D64.3 (VSS), D65.3 (VSS)
- net JTAG_SWO_TDO: no longer D113.2 (A), D118.2 (A), D122.2 (A), D4.2 (A), D69.2 (A), D73.2 (A), D78.2 (A), D9.2 (A), D91.2 (A)
- net VBUSOUT: now also D127.1 (VDD), D132.1 (VDD), D137.1 (VDD), D142.1 (VDD), D147.1 (VDD), D152.1 (VDD), D157.1 (VDD), D162.1 (VDD), D167.1 (VDD), D172.1 (VDD), D177.1 (VDD), D182.1 (VDD), D187.1 (VDD), D10.1 (VDD), D108.1 (VDD), D11.1 (VDD), D12.1 (VDD), D13.1 (VDD), D14.1 (VDD), D15.1 (VDD), D16.1 (VDD), D17.1 (VDD), D18.1 (VDD), D19.1 (VDD), D20.1 (VDD), D21.1 (VDD), D22.1 (VDD), D23.1 (VDD), D24.1 (VDD), D25.1 (VDD), D26.1 (VDD), D27.1 (VDD), D28.1 (VDD), D29.1 (VDD), D30.1 (VDD), D31.1 (VDD), D32.1 (VDD), D33.1 (VDD), D34.1 (VDD), D35.1 (VDD), D36.1 (VDD), D37.1 (VDD), D38.1 (VDD), D39.1 (VDD), D40.1 (VDD), D41.1 (VDD), D42.1 (VDD), D43.1 (VDD), D44.1 (VDD), D45.1 (VDD), D46.1 (VDD), D47.1 (VDD), D48.1 (VDD), D49.1 (VDD), D50.1 (VDD), D51.1 (VDD), D52.1 (VDD), D53.1 (VDD), D54.1 (VDD), D55.1 (VDD), D58.1 (VDD), D62.1 (VDD), D63.1 (VDD), D64.1 (VDD), D65.1 (VDD)
- net col0: no longer K01.1, K64.1, K65.1, K66.1, K67.1
- net col1: no longer K4.1, K68.1, K69.1, K70.1, K71.1
- net col11: no longer K112.1, K113.1, K114.1, K115.1, K116.1
- net col12: no longer K117.1, K118.1, K120.1, K5.1, K6.1
- net col13: no longer K122.1, K123.1, K124.1, K2.1, K3.1
- net col2: no longer K72.1, K73.1, K74.1, K75.1, K76.1
- net col3: no longer K77.1, K78.1, K79.1, K80.1
- net col4: no longer K81.1, K82.1, K83.1, K84.1
- net col5: no longer K85.1, K86.1, K87.1, K88.1, K89.1
- net col6: no longer K90.1, K91.1, K92.1, K93.1
- net col7: no longer K94.1, K95.1, K96.1, K97.1
- net col8: no longer K100.1, K101.1, K98.1, K99.1
- net col9: no longer K102.1, K103.1, K104.1, K105.1, K7.1
- net row0: no longer D1.2 (A), D100.2 (A), D104.2 (A), D109.2 (A), D114.2 (A), D119.2 (A), D123.2 (A), D70.2 (A), D74.2 (A), D79.2 (A), D83.2 (A), D87.2 (A), D92.2 (A), D96.2 (A)
- net row1: no longer D101.2 (A), D105.2 (A), D115.2 (A), D120.2 (A), D124.2 (A), D5.2 (A), D66.2 (A), D71.2 (A), D75.2 (A), D80.2 (A), D84.2 (A), D88.2 (A), D93.2 (A), D97.2 (A)
- net row2: no longer D102.2 (A), D106.2 (A), D111.2 (A), D116.2 (A), D125.2 (A), D67.2 (A), D7.2 (A), D72.2 (A), D76.2 (A), D81.2 (A), D85.2 (A), D89.2 (A), D94.2 (A), D98.2 (A)
- net row3: no longer D103.2 (A), D107.2 (A), D112.2 (A), D117.2 (A), D126.2 (A), D6.2 (A), D68.2 (A), D77.2 (A), D8.2 (A), D82.2 (A), D86.2 (A), D90.2 (A), D95.2 (A), D99.2 (A)
- net at D127.2 (DOUT): now also D132.4 (DIN)
- net ROW0_LED: now reaches D127.4 (DIN)
- net at D147.2 (DOUT): now also D152.4 (DIN)
- net at D147.4 (DIN): now also D142.2 (DOUT)
- net COL10: now reaches K107.1, K108.1, K109.1, K110.1, K111.1
- net at D132.2 (DOUT): now also D137.4 (DIN)
- net at D187.2 (DOUT): now also D23.4 (DIN)
- net at D187.4 (DIN): now also D182.2 (DOUT)
- net at D177.2 (DOUT): now also D182.4 (DIN)
- net at D177.4 (DIN): now also D172.2 (DOUT)
- net at D167.2 (DOUT): now also D172.4 (DIN)
- net at D167.4 (DIN): now also D162.2 (DOUT)
- net at D137.2 (DOUT): now also D142.4 (DIN)
- net at D162.4 (DIN): now also D157.2 (DOUT)
- net at D152.2 (DOUT): now also D157.4 (DIN)
- net P0.01/XL2 renamed ROW1_LED
- net ROW1_LED: now also D10.4 (DIN)
- net P0.02/NFC1: no longer names the net of A1.1, CT1.2, CT3.2, U4.W1 (P0.02/NFC1)
- net P0.03/NFC2: no longer names the net of A1.2, CT2.1, CT4.1, U4.AA1 (P0.03/NFC2)
- net P0.04/AIN0 renamed ROW2_LED
- net ROW2_LED: now also D25.4 (DIN)
- net P0.05/AIN1 renamed ROW3_LED
- net ROW3_LED: now also D39.4 (DIN)
- net P0.06/AIN2 renamed ROW4_LED
- net ROW4_LED: now also D53.4 (DIN)
- net P0.07/AIN3: no longer names the net of U4.AD2 (P0.07/AIN3)
- net P0.08/TRACEDATA3: no longer names the net of U4.AH2 (P0.08/TRACEDATA[3])
- net P0.09/TRACEDATA2: no longer names the net of U4.AJ1 (P0.09/TRACEDATA[2])
- net P0.10/TRACEDATA1: no longer names the net of U4.AK2 (P0.10/TRACEDATA[1])
- net P0.11/TRACEDATA0: no longer names the net of U4.AK4 (P0.11/TRACEDATA[0])
- net P0.12/TRACECLK: no longer names the net of U4.AK6 (P0.12/TRACECLK)
- net P0.13/QSPI0: no longer names the net of U4.AL5 (P0.13/QSPI[0])
- net P0.14/QSPI1: no longer names the net of U4.AK8 (P0.14/QSPI[1])
- net P0.15/QSPI2: no longer names the net of U4.AK10 (P0.15/QSPI[2])
- net P0.16/QSPI3: no longer names the net of U4.AL9 (P0.16/QSPI[3])
- net P0.17/QSPI_CLK: no longer names the net of U4.AK12 (P0.17/QSPI_CLK)
- net P0.18/QSPI_CS: no longer names the net of U4.AK14 (P0.18/QSPI_CS)
- net P0.19: no longer names the net of U4.AL13 (P0.19)
- net P0.20: no longer names the net of U4.AK16 (P0.20)
- net P0.21: no longer names the net of U4.AL15 (P0.21)
- net P0.22: no longer names the net of U4.AK18 (P0.22)
- net P0.23: no longer names the net of U4.AK20 (P0.23)
- net P0.24: no longer names the net of U4.AL27 (P0.24)
- net P0.25/AIN4: no longer names the net of U4.AK28 (P0.25/AIN4)
- net P0.26/AIN5: no longer names the net of U4.AL29 (P0.26/AIN5)
- net P0.27/AIN6: no longer names the net of U4.AK30 (P0.27/AIN6)
- net P0.28/AIN7: no longer names the net of U4.AE31 (P0.28/AIN7)
- net P0.29: no longer names the net of U4.U31 (P0.29)
- net P0.30: no longer names the net of U4.B24 (P0.30)
- net P0.31: no longer names the net of U4.B22 (P0.31)
- net P1.00: no longer names the net of U4.M2 (P1.00)
- net P1.01: no longer names the net of U4.P2 (P1.01)
- net P1.02/TWI: no longer names the net of U4.AE1 (P1.02/TWI)
- net P1.03/TWI: no longer names the net of U4.AF2 (P1.03/TWI)
- net P1.04: no longer names the net of U4.AL19 (P1.04)
- net P1.05: no longer names the net of U4.AK22 (P1.05)
- net P1.06: no longer names the net of U4.AL21 (P1.06)
- net P1.07: no longer names the net of U4.AK24 (P1.07)
- net P1.08: no longer names the net of U4.AL23 (P1.08)
- net P1.09: no longer names the net of U4.AK26 (P1.09)
- net P1.10: no longer names the net of U4.R31 (P1.10)
- net P1.11: no longer names the net of U4.B20 (P1.11)
- net P1.12: no longer names the net of U4.B18 (P1.12)
- net P1.13: no longer names the net of U4.A17 (P1.13)
- net P1.14: no longer names the net of U4.B16 (P1.14)
- net P1.15: no longer names the net of U4.B14 (P1.15)
- new net: D42.2 (DOUT), D43.4 (DIN)
- new net: D41.2 (DOUT), D42.4 (DIN)
- new net: D15.2 (DOUT), D16.4 (DIN)
- new net: D14.2 (DOUT), D15.4 (DIN)
- new net: D13.2 (DOUT), D14.4 (DIN)
- new net: D49.2 (DOUT), D50.4 (DIN)
- new net: D48.2 (DOUT), D49.4 (DIN)
- new net: D37.2 (DOUT), D38.4 (DIN)
- new net: D36.2 (DOUT), D37.4 (DIN)
- new net: D33.2 (DOUT), D34.4 (DIN)
- new net: D32.2 (DOUT), D33.4 (DIN)
- new net: D63.2 (DOUT), D64.4 (DIN)
- new net: D62.2 (DOUT), D63.4 (DIN)
- new net: D28.2 (DOUT), D29.4 (DIN)
- new net: D27.2 (DOUT), D28.4 (DIN)
- new net: D26.2 (DOUT), D27.4 (DIN)
- new net: D21.2 (DOUT), D22.4 (DIN)
- new net: D20.2 (DOUT), D21.4 (DIN)
- new net: D19.2 (DOUT), D20.4 (DIN)
- new net: D18.2 (DOUT), D19.4 (DIN)
- new net: D47.2 (DOUT), D48.4 (DIN)
- new net: D35.2 (DOUT), D36.4 (DIN)
- new net: D53.2 (DOUT), D54.4 (DIN)
- new net: D17.2 (DOUT), D18.4 (DIN)
- new net: D16.2 (DOUT), D17.4 (DIN)
- new net: D25.2 (DOUT), D26.4 (DIN)
- new net: D51.2 (DOUT), D52.4 (DIN)
- new net: D50.2 (DOUT), D51.4 (DIN)
- new net: D46.2 (DOUT), D47.4 (DIN)
- new net: D12.2 (DOUT), D13.4 (DIN)
- new net: D108.4 (DIN), D65.2 (DOUT)
- new net: D55.2 (DOUT), D58.4 (DIN)
- new net: D54.2 (DOUT), D55.4 (DIN)
- new net: D40.2 (DOUT), D41.4 (DIN)
- new net: D45.2 (DOUT), D46.4 (DIN)
- new net: D64.2 (DOUT), D65.4 (DIN)
- new net: D43.2 (DOUT), D44.4 (DIN)
- new net: D34.2 (DOUT), D35.4 (DIN)
- new net: D10.2 (DOUT), D11.4 (DIN)
- new net: D22.2 (DOUT), D24.4 (DIN)
- new net: D11.2 (DOUT), D12.4 (DIN)
- new net: D44.2 (DOUT), D45.4 (DIN)
- new net: D58.2 (DOUT), D62.4 (DIN)
- new net: D39.2 (DOUT), D40.4 (DIN)
- new net: D30.2 (DOUT), D31.4 (DIN)
- new net: D29.2 (DOUT), D30.4 (DIN)
- new net: D31.2 (DOUT), D32.4 (DIN)
- new net COL0: K01.1, K64.1, K65.1, K66.1, K67.1
- new net COL1: K4.1, K68.1, K69.1, K70.1, K71.1
- new net COL11: K112.1, K113.1, K114.1, K115.1, K116.1
- new net COL12: K117.1, K118.1, K120.1, K5.1, K6.1
- new net COL13: K122.1, K123.1, K124.1, K2.1, K3.1
- new net COL2: K72.1, K73.1, K74.1, K75.1, K76.1
- new net COL3: K77.1, K78.1, K79.1, K80.1
- new net COL4: K81.1, K82.1, K83.1, K84.1
- new net COL5: K85.1, K86.1, K87.1, K88.1, K89.1
- new net COL6: K90.1, K91.1, K92.1, K93.1
- new net COL7: K94.1, K95.1, K96.1, K97.1
- new net COL8: K100.1, K101.1, K98.1, K99.1
- new net COL9: K102.1, K103.1, K104.1, K105.1, K7.1
- new net ROW0: D1.2 (A), D100.2 (A), D104.2 (A), D109.2 (A), D114.2 (A), D119.2 (A), D123.2 (A), D70.2 (A), D74.2 (A), D79.2 (A), D83.2 (A), D87.2 (A), D92.2 (A), D96.2 (A)
- new net ROW1: D101.2 (A), D105.2 (A), D115.2 (A), D120.2 (A), D124.2 (A), D5.2 (A), D66.2 (A), D71.2 (A), D75.2 (A), D80.2 (A), D84.2 (A), D88.2 (A), D93.2 (A), D97.2 (A)
- new net ROW2: D102.2 (A), D106.2 (A), D111.2 (A), D116.2 (A), D125.2 (A), D67.2 (A), D7.2 (A), D72.2 (A), D76.2 (A), D81.2 (A), D85.2 (A), D89.2 (A), D94.2 (A), D98.2 (A)
- new net ROW3: D103.2 (A), D107.2 (A), D112.2 (A), D117.2 (A), D126.2 (A), D6.2 (A), D68.2 (A), D77.2 (A), D8.2 (A), D82.2 (A), D86.2 (A), D90.2 (A), D95.2 (A), D99.2 (A)
- new net ROW4: D113.2 (A), D118.2 (A), D122.2 (A), D4.2 (A), D69.2 (A), D73.2 (A), D78.2 (A), D9.2 (A), D91.2 (A)
Other:
- note added: "0"
- note added: "1"
- note added: "2"
- note added: "3"
- note added: "4"
- note added: "5"
- note added: "6"
- note added: "7"
- note added: "8"
- note added: "9"
- note added: "A"
- note added: "B"
- note added: "BACKSLASH"
- note added: "BACKSPACE"
- note added: "C"
- note added: "CAPSLOCK"
- note added: "COMMA"
- note added: "D"
- note added: "DOWN"
- note added: "E"
- note added: "ENTER"
- note added: "EQUALS"
- note added: "ESC"
- note added: "F"
- note added: "FN"
- note added: "FSLASH"
- note added: "G"
- note added: "H"
- note added: "I"
- note added: "J"
- note added: "K"
- note added: "L"
- note added: "LALT"
- note added: "LCTRL"
- note added: "LEFT"
- note added: "LSHIFT"
- note added: "M"
- note added: "MENU"
- note added: "MINUS"
- note added: "N"
- note added: "O"
- note added: "P"
- note added: "PERIOD"
- note added: "Q"
- note added: "QUOTE"
- note added: "R"
- note added: "RALT"
- note added: "RCTRL"
- note added: "RIGHT"
- note added: "RSHIFT"
- note added: "S"
- note added: "SEMICOLON"
- note added: "SPACE"
- note added: "T"
- note added: "TAB"
- note added: "U"
- note added: "UP"
- note added: "V"
- note added: "W"
- note added: "WIN"
- note added: "X"
- note added: "Y"
- note added: "Z"
- note added: "["
- note added: "]"
- note removed: "Optional"
- moved on the sheet: A1, CT2, CT3, CT4

Commit message: Added macro column and possible rotary encoder
Parts:
- added D110, D121, D128, D129, D130: WS2812B, LED_SMD:LED_WS2812B_PLCC4_5.0x5.0mm_P3.2mm, symbol LED:WS2812B
- added D56, D57, D59, D60, D61: D, Diode_SMD:D_SOD-123, symbol Device:D
- added K10: KEYSW, MX_Hotswap:MX-Hotswap-2.25U, symbol keyboard_parts:KEYSW
- added K11, K12: KEYSW, MX_Hotswap:MX-Hotswap-1.25U, symbol keyboard_parts:KEYSW
- added K8, K9: KEYSW, MX_Hotswap:MX-Hotswap-1.5U, symbol keyboard_parts:KEYSW
Connections:
- net COL0: now also U4.B14 (P1.15)
- net COL1: now also U4.AL13 (P0.19)
- net COL10: now also U4.AE31 (P0.28/AIN7)
- net COL11: now also U4.U31 (P0.29)
- net COL12: now also U4.B24 (P0.30)
- net COL13: now also U4.B22 (P0.31)
- net COL2: now also U4.AK16 (P0.20)
- net COL3: now also U4.AL15 (P0.21)
- net COL4: now also U4.AK18 (P0.22)
- net COL5: now also U4.AK20 (P0.23)
- net COL6: now also U4.AL27 (P0.24)
- net COL7: now also U4.AK28 (P0.25/AIN4)
- net COL8: now also U4.AL29 (P0.26/AIN5)
- net COL9: now also U4.AK30 (P0.27/AIN6)
- net GND: now also D110.3 (VSS), D121.3 (VSS), D128.3 (VSS), D129.3 (VSS), D130.3 (VSS)
- net LCD_DC: now also U4.AK6 (P0.12/TRACECLK)
- net LCD_MISO: now also U4.AK2 (P0.10/TRACEDATA[1])
- net LCD_MOSI: now also U4.AJ1 (P0.09/TRACEDATA[2])
- net LCD_Reset: now also U4.AK22 (P1.05)
- net LCD_clk: now also U4.AH2 (P0.08/TRACEDATA[3])
- net LCD_fs: now also U4.AK4 (P0.11/TRACEDATA[0])
- net ROW0: now also U4.AD2 (P0.07/AIN3), D56.2 (A)
- net ROW1: now also U4.B20 (P1.11), D57.2 (A)
- net ROW2: now also U4.B18 (P1.12), D59.2 (A)
- net ROW3: now also U4.A17 (P1.13), D60.2 (A)
- net ROW4: now also U4.B16 (P1.14), D61.2 (A)
- net VBUSOUT: now also D110.1 (VDD), D121.1 (VDD), D128.1 (VDD), D129.1 (VDD), D130.1 (VDD)
- net ~{BLUETOOTH_LED}: now also U4.AK24 (P1.07)
- net ~{CAPS_LOCK_LED}: now also U4.AL21 (P1.06)
- net ENC_B: now reaches U4.AK26 (P1.09)
- net ENC_A: now reaches U4.AL23 (P1.08)
- net COL14: now reaches U4.R31 (P1.10)
- net COL14: now also K10.1, K11.1, K12.1, K8.1, K9.1
- net at D23.2 (DOUT): now also D110.4 (DIN)
- net at D108.2 (DOUT): now also D130.4 (DIN)
- net at D52.2 (DOUT): now also D129.4 (DIN)
- net FLASH_2: now reaches U4.AK10 (P0.15/QSPI[2])
- net FLASH_CLK: now reaches U4.AK12 (P0.17/QSPI_CLK)
- net FLASH_CS: now reaches U4.AK14 (P0.18/QSPI_CS)
- net FLASH_1: now reaches U4.AK8 (P0.14/QSPI[1])
- net FLASH_0: now reaches U4.AL5 (P0.13/QSPI[0])
- net FLASH_3: now reaches U4.AL9 (P0.16/QSPI[3])
- net at D24.2 (DOUT): now also D121.4 (DIN)
- net at D38.2 (DOUT): now also D128.4 (DIN)
- new net: D56.1 (K), K8.2
- new net: D59.1 (K), K10.2
- new net: D57.1 (K), K9.2
- new net: D60.1 (K), K11.2
- new net: D61.1 (K), K12.2
Other:
- note added: "MACRO1"
- note added: "MACRO2"
- note added: "MACRO3"
- note added: "MACRO4"
- note added: "MACRO5"

Commit message: Every day God abandons me
Parts:
- removed C10, C12, C14, C15, C3, C8: 0.1u, Capacitor_SMD:C_0603_1608Metric_Pad1.08x0.95mm_HandSolder, symbol Device:C
- removed C13, C4: 10p, Capacitor_SMD:C_0603_1608Metric_Pad1.08x0.95mm_HandSolder, symbol Device:C
- removed C16: 0.01u, Capacitor_SMD:C_0603_1608Metric_Pad1.08x0.95mm_HandSolder, symbol Device:C
- removed C2, C9: 1.0u, Capacitor_SMD:C_0603_1608Metric_Pad1.08x0.95mm_HandSolder, symbol Device:C
- removed C5: 2.2u, Capacitor_SMD:C_0603_1608Metric_Pad1.08x0.95mm_HandSolder, symbol Device:C
- removed D2, D3: LED, LED_SMD:LED_0603_1608Metric_Pad1.05x0.95mm_HandSolder, symbol Device:LED
- removed IC2: BGM220PC22HNA2R, BluetoothModuleLibrary:BGM220PC22HNA2R, symbol BGM220PC22HNA2R:BGM220PC22HNA2R
- removed J4: USB_B_Micro, Connector_USB:USB_Micro-B_Amphenol_10103594-0001LF_Horizontal, symbol Connector:USB_B_Micro
- removed LD1: ${ALTIUM_VALUE}, LED_RGB_0603, symbol npm1300_qeaa_config1-altium-import:root_0_D{colon}LED_RGB
- removed R2: 10k, Resistor_SMD:R_0402_1005Metric, symbol Device:R
- removed R3: 330, Resistor_SMD:R_0402_1005Metric, symbol Device:R
- removed R5, R6: 22, Resistor_SMD:R_0402_1005Metric, symbol Device:R
- removed R7, R8: 1.1k, Resistor_SMD:R_0402_1005Metric, symbol Device:R
- removed TP4: GND, TestPoint:TestPoint_Pad_2.5x2.5mm, symbol Connector:TestPoint
- removed U3: TM4C123GH6PMI7, TM4C:QFP50P1200X1200X160-64N, symbol TM4C123GH6PM:TM4C123GH6PMI7
- removed X1: 16MHz, CrystalLibrary:NX5032GA16000000MHZLNCD1, symbol keyboard_parts:XTAL
- added IC1, IC3: SN74HC251PWR, SOP65P640X120-16N, symbol SN74HC251PWR:SN74HC251PWR
- added IC2: SN74LV138APWR, SOP65P640X120-16N, symbol SN74LV138APWR:SN74LV138APWR
- added R1, R4: 22, Resistor_SMD:R_0402_1005Metric, symbol Device:R
- added SW1: RotaryEncoder_Switch, symbol Device:RotaryEncoder_Switch
- added U2: VEML6030, VEML6030:Vishay-6.550-5348.01-4-02_2016-1-MFG, symbol eec:VEML6030
- C19, C20, C22, C26, C27: footprint CAPC1005X04L -> Capacitor_SMD:C_0603_1608Metric_Pad1.08x0.95mm_HandSolder
- C21, C23, C38, C39, C41, C42, C43, C44, C45, C46, C47, C48, C49, C50: footprint CAPC1608X06L -> Capacitor_SMD:C_0603_1608Metric_Pad1.08x0.95mm_HandSolder
- C24, C25, C28, C29, C30, C31, C32, C33, C34, C35, C36, C40, CT1, CT2, CT3, CT4: footprint CAPC0603X03L_C -> Capacitor_SMD:C_0603_1608Metric_Pad1.08x0.95mm_HandSolder
- C37: footprint CAPC0603X03L_C_NC -> Capacitor_SMD:C_0603_1608Metric_Pad1.08x0.95mm_HandSolder
- J2: footprint (none) -> Connector_PinHeader_2.54mm:PinHeader_2x05_P2.54mm_Vertical
- J7: footprint TP_3x1mm_TH -> Connector_JST:JST_EH_B2B-EH-A_1x02_P2.50mm_Vertical
- L1, L2: footprint INDC1608X06L -> Inductor_SMD:L_0805_2012Metric_Pad1.15x1.40mm_HandSolder
- L3: footprint INDC0603X03L_C -> Inductor_SMD:L_0805_2012Metric_Pad1.15x1.40mm_HandSolder
- L4, L5: footprint INDC2016X10N -> Inductor_SMD:L_0805_2012Metric_Pad1.15x1.40mm_HandSolder
- R10, R11, R12, R13, R9: footprint RESC0603X03L_C -> Resistor_SMD:R_0603_1608Metric_Pad0.98x0.95mm_HandSolder
- U4: footprint AQFN40P700X700X85_HS-99N -> nRF5340-QKAA:Nordic_Semiconductor-NRF5340-QKAA-R7-MFG
- U5: footprint Nordic_QFN50P500X500X90-33N -> nPM1300:nPM1300-QEAA
- X3: footprint BT-XTAL_2016 -> Crystal:Crystal_SMD_MicroCrystal_CC1V-T1A-2Pin_8.0x3.7mm_HandSoldering
Connections:
- net GPIO0 is gone; now on net NPM_INT: U5.7 (GPIO0)
- net GPIO1 is gone; now on net ~{RESET}: U5.8 (GPIO1)
- net JTAG_SWCLK_TCLK is gone; now on net SWDCLK: J2.4 (SWDCLK/TCK)
- net JTAG_SWDIO_TMS is gone; now on net SWDIO: J2.2 (SWDIO/TMS)
- net SCL is gone; now on net NPM_SCL: R12.1, U5.14 (SCL)
- net SDA is gone; now on net NPM_SDA: R13.1, U5.13 (SDA)
- net 3V3: now also IC1.16 (VCC), IC2.16 (VCC), IC3.16 (VCC), SW1.C, SW1.S1, U2.6 (VDD); no longer U1.1 (LITE)
- net CC1: now also J1.A5 (CC1)
- net CC2: now also J1.B5 (CC2)
- net COL0: now also IC1.4 (D0); no longer U4.B14 (P1.15)
- net COL1: now also IC1.3 (D1); no longer U4.AL13 (P0.19)
- net COL10: now also IC3.2 (D2); no longer U4.AE31 (P0.28/AIN7)
- net COL11: now also IC3.1 (D3); no longer U4.U31 (P0.29)
- net COL12: now also IC3.15 (D4); no longer U4.B24 (P0.30)
- net COL13: now also IC3.14 (D5); no longer U4.B22 (P0.31)
- net COL14: now also IC3.13 (D6); no longer U4.R31 (P1.10)
- net COL2: now also IC1.2 (D2); no longer U4.AK16 (P0.20)
- net COL3: now also IC1.1 (D3); no longer U4.AL15 (P0.21)
- net COL4: now also IC1.15 (D4); no longer U4.AK18 (P0.22)
- net COL5: now also IC1.14 (D5); no longer U4.AK20 (P0.23)
- net COL6: now also IC1.13 (D6); no longer U4.AL27 (P0.24)
- net COL7: now also IC1.12 (D7); no longer U4.AK28 (P0.25/AIN4)
- net COL8: now also IC3.4 (D0); no longer U4.AL29 (P0.26/AIN5)
- net COL9: now also IC3.3 (D1); no longer U4.AK30 (P0.27/AIN6)
- net D_N: now also R1.2
- net D_P: now also R4.2
- net ENC_A: now also U4.M2 (P1.00), SW1.A; no longer U4.AL23 (P1.08)
- net ENC_B: now also U4.P2 (P1.01), SW1.B; no longer U4.AK26 (P1.09)
- net GND: now also J1.A1 (GND), J1.A12 (GND), J1.B1 (GND), J1.B12 (GND), J1.S1 (SHIELD), IC1.7 (~{OE}), IC1.8 (GND), IC2.4 (~{G0}), IC2.5 (~{G1}), IC2.8 (GND), IC3.12 (D7), IC3.7 (~{OE}), IC3.8 (GND), U2.1 (GND), U2.4 (ADDR)
- net ROW0: now also IC2.15 (Y0); no longer U4.AD2 (P0.07/AIN3)
- net ROW1: now also IC2.14 (Y1); no longer U4.B20 (P1.11)
- net ROW2: now also IC2.13 (Y2); no longer U4.B18 (P1.12)
- net ROW3: now also IC2.12 (Y3); no longer U4.A17 (P1.13)
- net ROW4: now also IC2.11 (Y4); no longer U4.B16 (P1.14)
- net VBUSIN: now also J1.A4 (VBUS), J1.A9 (VBUS), J1.B4 (VBUS), J1.B9 (VBUS)
- net NPM_SCL: now reaches U4.AE1 (P1.02/TWI)
- net NPM_SDA: now reaches U4.AF2 (P1.03/TWI)
- net NPM_INT: now reaches U4.AL19 (P1.04)
- net at J1.A6 (D+): now also J1.B6 (D+), R4.1
- net at J1.A7 (D-): now also J1.B7 (D-), R1.1
- net GPIO2: no longer names the net of U5.9 (GPIO2)
- net GPIO3: no longer names the net of U5.10 (GPIO3)
- net GPIO4: no longer names the net of U5.11 (GPIO4)
- net JTAG_SWO_TDO: no longer names the net of J2.6 (SWO/TDO)
- net JTAG_TDI: no longer names the net of J2.8 (NC/TDI)
- net LED0: no longer names the net of U5.25 (LED0)
- net LED1: no longer names the net of U5.26 (LED1)
- net LED2: no longer names the net of U5.27 (LED2)
- net ~{BLUETOOTH_LED} renamed LIGHT_SCL
- net LIGHT_SCL: now also U2.5 (SCL)
- net ~{CAPS_LOCK_LED} renamed LCD_LITE
- net LCD_LITE: now also U1.1 (LITE)
- new net COLMUX_A: IC1.11 (A), IC3.11 (A)
- new net COLMUX_B: IC1.10 (B), IC3.10 (B)
- new net COLMUX_C: IC1.9 (C), IC3.9 (C)
- new net COLMUX_OUTA: IC1.5 (Y)
- new net COLMUX_OUTB: IC3.5 (Y)
- new net ENC_SW: SW1.S2, U4.AK26 (P1.09)
- new net LIGHT_SDA: U2.2 (SDA), U4.AL23 (P1.08)
- new net ROWDEMUX_A: IC2.1 (A)
- new net ROWDEMUX_B: IC2.2 (B)
- new net ROWDEMUX_C: IC2.3 (C)
- no-connect marks 16 -> 19
Other:
- note added: "COLMUX_D = 0 -> Cols 0-7 COLMUX_D = 1 -> Cols 8-14"
- note removed: "Already pulled by ICDI TM4C"
- note removed: "C14 should be placed on pin 25 C11/12/13 on pin 56"
- note removed: "ID Grounded = HOST ID Floating = DEVICE"
- note removed: "No reset switch necessary Just toggle the power (switch or JTAG)"
- note removed: "PB2 is BGM220P RX PB1 is BGM220P TX BLUETOOTH_?X is relative to the TM4C"
- note removed: "Place a .1uF cap on each VDD pin 1uF and 10nF caps isolate VDD from VDDA"
- note removed: "See 24.9.5 in the datasheet"
- note removed: "See Table 23-7 in the TM4C123 datasheet"
- note removed: "USB series resistors are ??? ripped from an example KB schematic probably just need to ensure 90 ohm diff impedance"
- note removed: "Verified"
- moved on the sheet: A1, CT2, CT3, CT4
