File: hw/PCB/PCB.kicad_sch (KiCad schematic)
At the start: 273 parts, among them IC1 SN74HC251PWR, IC2 SN74LV138APWR, IC3 SN74HC251PWR, J1 USB_C_Receptacle_USB2.0, J2 Conn_ARM_JTAG_SWD_10, J7 ${ALTIUM_VALUE}, K01 KEYSW, K10 KEYSW, K100 KEYSW, K101 KEYSW, K102 KEYSW, K103 KEYSW, K104 KEYSW, K105 KEYSW, K107 KEYSW, K108 KEYSW, K109 KEYSW, K11 KEYSW, K110 KEYSW, K111 KEYSW, K112 KEYSW, K113 KEYSW, K114 KEYSW, K115 KEYSW, K116 KEYSW, K117 KEYSW, K118 KEYSW, K12 KEYSW, K120 KEYSW, K122 KEYSW, K123 KEYSW, K124 KEYSW, K2 KEYSW, K3 KEYSW, K4 KEYSW, K5 KEYSW, K6 KEYSW, K64 KEYSW, K65 KEYSW, K66 KEYSW, K67 KEYSW, K68 KEYSW, K69 KEYSW, K7 KEYSW, K70 KEYSW, K71 KEYSW, K72 KEYSW, K73 KEYSW, K74 KEYSW, K75 KEYSW, K76 KEYSW, K77 KEYSW, K78 KEYSW, K79 KEYSW, K8 KEYSW, K80 KEYSW, K81 KEYSW, K82 KEYSW, K83 KEYSW, K84 KEYSW, K85 KEYSW, K86 KEYSW, K87 KEYSW, K88 KEYSW, K89 KEYSW, K9 KEYSW, K90 KEYSW, K91 KEYSW, K92 KEYSW, K93 KEYSW, K94 KEYSW, K95 KEYSW, K96 KEYSW, K97 KEYSW, K98 KEYSW, K99 KEYSW, SW1 RotaryEncoder_Switch, U1 Adafruit ST7735R, U2 VEML6030, U4 ${ALTIUM_VALUE}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

Commit message: Blocked out connections of the peripherals to the STM32L552
Parts:
- removed A1: ${ALTIUM_VALUE}, TP_2x1mm_TH, symbol nrf5340_qkaa_config2-altium-import:root_3_mirrored_NFC_Antenna
- removed C19, C21, C23, C24, C25, C28, C29, C30, C31, C33, C34, C35, C36: ${ALTIUM_VALUE}, Capacitor_SMD:C_0603_1608Metric_Pad1.08x0.95mm_HandSolder, symbol nrf5340_qkaa_config2-altium-import:root_3_CAP
- removed C20, C22, C26, C27, C32, C37: ${ALTIUM_VALUE}, Capacitor_SMD:C_0603_1608Metric_Pad1.08x0.95mm_HandSolder, symbol nrf5340_qkaa_config2-altium-import:root_1_CAP
- removed C38, C39, C41, C42, C43, C44, C45, C46, C47, C48, C49, C50: ${ALTIUM_VALUE}, Capacitor_SMD:C_0603_1608Metric_Pad1.08x0.95mm_HandSolder, symbol npm1300_qeaa_config1-altium-import:root_1_CAP
- removed C40: ${ALTIUM_VALUE}, Capacitor_SMD:C_0603_1608Metric_Pad1.08x0.95mm_HandSolder, symbol npm1300_qeaa_config1-altium-import:root_3_CAP
- removed CT1, CT2, CT3, CT4: ${ALTIUM_VALUE}, Capacitor_SMD:C_0603_1608Metric_Pad1.08x0.95mm_HandSolder, symbol nrf5340_qkaa_config2-altium-import:root_3_mirrored_CAP
- removed J7: ${ALTIUM_VALUE}, Connector_JST:JST_EH_B2B-EH-A_1x02_P2.50mm_Vertical, symbol npm1300_qeaa_config1-altium-import:root_0_Battery_pack_NTC
- removed L1, L2: ${ALTIUM_VALUE}, Inductor_SMD:L_0805_2012Metric_Pad1.15x1.40mm_HandSolder, symbol nrf5340_qkaa_config2-altium-import:root_1_IND
- removed L3: ${ALTIUM_VALUE}, Inductor_SMD:L_0805_2012Metric_Pad1.15x1.40mm_HandSolder, symbol nrf5340_qkaa_config2-altium-import:root_0_mirrored_IND
- removed L4, L5: ${ALTIUM_VALUE}, Inductor_SMD:L_0805_2012Metric_Pad1.15x1.40mm_HandSolder, symbol npm1300_qeaa_config1-altium-import:root_3_IND
- removed R10, R11: ${ALTIUM_VALUE}, Resistor_SMD:R_0603_1608Metric_Pad0.98x0.95mm_HandSolder, symbol npm1300_qeaa_config1-altium-import:root_3_mirrored_RES
- removed R12, R13: ${ALTIUM_VALUE}, Resistor_SMD:R_0603_1608Metric_Pad0.98x0.95mm_HandSolder, symbol npm1300_qeaa_config1-altium-import:root_3_RES
- removed R9: ${ALTIUM_VALUE}, Resistor_SMD:R_0603_1608Metric_Pad0.98x0.95mm_HandSolder, symbol nrf5340_qkaa_config2-altium-import:root_0_RES
- removed U4: ${ALTIUM_VALUE}, nRF5340-QKAA:Nordic_Semiconductor-NRF5340-QKAA-R7-MFG, symbol nrf5340_qkaa_config2-altium-import:root_0_nRF5340_QKAA
- removed U5: ${ALTIUM_VALUE}, nPM1300:nPM1300-QEAA, symbol npm1300_qeaa_config1-altium-import:root_0_nPM1300_QEAA
- removed X3: ${ALTIUM_VALUE}, Crystal:Crystal_SMD_MicroCrystal_CC1V-T1A-2Pin_8.0x3.7mm_HandSoldering, symbol nrf5340_qkaa_config2-altium-import:root_1_XTAL_4-pin_grounded
- added BT1, BT2, BT3: 1.5V, symbol BA1AAPC:BA1AAPC
- added C1, C2: 0.1u, Capacitor_SMD:C_0603_1608Metric_Pad1.08x0.95mm_HandSolder, symbol Device:C
- added C3: 1.0u, Capacitor_SMD:C_0603_1608Metric_Pad1.08x0.95mm_HandSolder, symbol Device:C
- added C4: 0.01u, Capacitor_SMD:C_0603_1608Metric_Pad1.08x0.95mm_HandSolder, symbol Device:C
- added D2: LED, LED_SMD:LED_0603_1608Metric_Pad1.05x0.95mm_HandSolder, symbol Device:LED
- added IC4: BGM220PC22HNA2R, BluetoothModuleLibrary:BGM220PC22HNA2R, symbol BGM220PC22HNA2R:BGM220PC22HNA2R
- added IC5: TPS2113ADRBR, SwitchingICLibrary:SON65P300X300X100-9N-D, symbol TPS2113ADRBR:TPS2113ADRBR
- added J3: Conn_02x05_Odd_Even, Connector_PinHeader_1.27mm:PinHeader_2x05_P1.27mm_Vertical, symbol Connector_Generic:Conn_02x05_Odd_Even
- added J4: BATT_POS, Connector_Pin:Pin_D1.0mm_L10.0mm, symbol Connector:Conn_01x01_Pin
- added J5: BATT_NEG, Connector_Pin:Pin_D1.0mm_L10.0mm, symbol Connector:Conn_01x01_Pin
- added R2, R3: 10k, Resistor_SMD:R_0402_1005Metric, symbol Device:R
- added R5: 750, Resistor_SMD:R_0402_1005Metric, symbol Device:R
- added R6: 1.1k, Resistor_SMD:R_0402_1005Metric, symbol Device:R
- added SW2: BAT_SWITCH, SLW-121586-5A-D:SLW1215865AD, symbol Switch:SW_SPDT
- added TP1: VBAT, TestPoint:TestPoint_Pad_2.5x2.5mm, symbol Connector:TestPoint
- added TP2: Switch_OUT, TestPoint:TestPoint_Pad_2.5x2.5mm, symbol Connector:TestPoint
- added TP3: IN1, TestPoint:TestPoint_Pad_2.5x2.5mm, symbol Connector:TestPoint
- added TP4: 3V3, TestPoint:TestPoint_Pad_2.5x2.5mm, symbol Connector:TestPoint
- added U3: STM32L552RETx, Package_QFP:LQFP-64_10x10mm_P0.5mm, symbol MCU_ST_STM32L5:STM32L552RETx
- added U4: S25FL127SABMFI101, SOC008_SPA, symbol 2023-12-04_00-10-28:S25FL127SABMFI101
- added U5: TPS73633DBV, Package_TO_SOT_SMD:SOT-23-5, symbol Regulator_Linear:TPS73633DBV
Connections:
- net VBUSIN is gone; now on net VBUS: J1.A4 (VBUS), J1.A9 (VBUS), J1.B4 (VBUS), J1.B9 (VBUS)
- net 3V3: now also IC4.13 (VDD), J3.1 (Pin_1), R2.1, R6.1, TP4.1, U4.8 (VCC), U5.5 (OUT)
- net COLMUX_A: now also U3.10 (PC2)
- net COLMUX_B: now also U3.11 (PC3)
- net COLMUX_C: now also U3.24 (PC4)
- net COLMUX_OUTA: now also U3.8 (PC0)
- net COLMUX_OUTB: now also U3.9 (PC1)
- net D_N: now also U3.44 (PA11)
- net D_P: now also U3.45 (PA12)
- net ENC_A: now also U3.14 (PA0)
- net ENC_B: now also U3.15 (PA1)
- net ENC_SW: now also U3.57 (PB5)
- net FLASH_0: now also U3.27 (PB1), U4.5 (SI/IO0)
- net FLASH_1: now also U3.26 (PB0), U4.2 (SO/IO1)
- net FLASH_2: now also U3.23 (PA7), U4.3 (*WP/IO2)
- net FLASH_3: now also U3.22 (PA6), U4.7 (*HOLD/IO3)
- net FLASH_CLK: now also U3.17 (PA3), U4.6 (CLK)
- net FLASH_CS: now also U3.16 (PA2), U4.1 (*CS)
- net GND: now also BT3.-, C1.2, C2.2, C3.1, C4.2, D2.1 (K), IC4.1 (GND_1), IC4.12 (GND_2), IC4.20 (GND_3), IC4.31 (GND_4), IC5.2 (~{EN}), IC5.3 (VSNS), IC5.5 (GND_1), IC5.9 (GND_2), J3.2 (Pin_2), J5.1 (Pin_1), R5.2, SW2.3 (C), U3.12 (VSSA), U3.18 (VSS), U3.31 (VSS), U3.47 (VSS), U3.63 (VSS), U4.4 (GND), U5.2 (GND)
- net LCD_DC: now also U3.30 (PB11)
- net LCD_LITE: now also U3.29 (PB10)
- net LCD_MISO: now also U3.35 (PB14)
- net LCD_MOSI: now also U3.36 (PB15)
- net LCD_Reset: now also U3.62 (PB9)
- net LCD_clk: now also U3.42 (PA9)
- net LCD_fs: now also U3.33 (PB12)
- net LIGHT_SCL: now also U3.58 (PB6)
- net LIGHT_SDA: now also U3.59 (PB7)
- net ROW0_LED: now also U3.39 (PC8)
- net ROW1_LED: now also U3.40 (PC9)
- net ROW2_LED: now also U3.53 (PC12)
- net ROW3_LED: now also U3.2 (PC13)
- net ROW4_LED: now also U3.61 (PB8)
- net ROWDEMUX_A: now also U3.25 (PC5)
- net ROWDEMUX_B: now also U3.37 (PC6)
- net ROWDEMUX_C: now also U3.38 (PC7)
- net VBAT: now also C1.1, IC5.6 (IN2), SW2.2 (B), TP1.1
- net VBUS: now also C2.1, IC5.8 (IN1), TP3.1
- net ~{RESET}: now also R3.2, U3.7 (NRST)
- net JTAG_TDO: now reaches J2.6 (SWO/TDO)
- net JTAG_TDO: now also U3.55 (PB3)
- net JTAG_TDI: now reaches J2.8 (NC/TDI)
- net JTAG_TDI: now also U3.50 (PA15)
- net LCD_SD_Card: no longer names the net of U1.6 (CARD_CS)
- net SWDCLK renamed JTAG_TCK
- net JTAG_TCK: now also U3.49 (PA14)
- net SWDIO renamed JTAG_TMS
- net JTAG_TMS: now also U3.46 (PA13)
- net VBUSOUT renamed Switch_OUT
- net Switch_OUT: now also C3.2, IC5.7 (OUT), TP2.1, U5.1 (IN), U5.3 (EN)
- new net: C4.1, U5.4 (NR)
- new net: R3.1, U3.1 (VBAT), U3.13 (VDDA), U3.19 (VDD), U3.32 (VDD), U3.48 (VDDUSB), U3.64 (VDD)
- new net: D2.2 (A), R6.2
- new net: BT1.-, BT2.+
- new net: BT2.-, BT3.+
- new net: IC5.4 (ILIM), R5.1
- new net: BT1.+, J4.1 (Pin_1), SW2.1 (A)
- new net BGM_SWCLK: IC4.8 (PA01), J3.8 (Pin_8)
- new net BGM_SWDIO: IC4.9 (PA02), J3.7 (Pin_7)
- new net BGM_SWO: IC4.10 (PA03), J3.6 (Pin_6)
- new net BLUETOOTH_CTS: IC4.16 (PA07), U3.34 (PB13)
- new net BLUETOOTH_RTS: IC4.17 (PA08), U3.54 (PD2)
- new net BLUETOOTH_RX: IC4.14 (PA05), U3.52 (PC11)
- new net BLUETOOTH_TX: IC4.15 (PA06), U3.51 (PC10)
- new net BLUETOOTH_~{RESET}: IC4.30 (RESETN), J3.3 (Pin_3), R2.2, U3.20 (PA4)
- new net EM4_WAKEUP: IC4.22 (PC00), U3.21 (PA5), U3.56 (PB4)
- new net PTI_DFRAME: IC4.27 (PC05), J3.9 (Pin_9)
- new net PTI_DOUT: IC4.26 (PC04), J3.10 (Pin_10)
- new net ~{BLUETOOTH_LED}: IC4.3 (PB03)
- no-connect marks 19 -> 34
Other:
- note added: "BLUETOOTH_?X/?TS are relative to the main MCU"
- note added: "I2C1_SCL"
- note added: "I2C1_SCL/USART1_TX"
- note added: "I2C1_SDA/SPI2_NSS"
- note added: "I2C1_SDA/USART1_RX"
- note added: "ILIM - Current Limit Current Limit = 500/R TPS2113A can do 630mA min limit R = 500/0.630 ~= 800 Ohm"
- note added: "JTAG_CLK/SWD_CLK/I2C1_SMBA"
- note added: "JTAG_TDI/SPI1_NSS/TIM2_CH1/TIM2_ETR/USART2_RX/USART3_RTS_DE/USB_CC1"
- note added: "JTAG_TDO/SWO/SPI1_SCK/TM2_CH2/USART1_RTS_DE"
- note added: "JTAG_TMS/SWDIO/USB_NOE"
- note added: "Must have a large copper ground pour to dissipate heat properly"
- note added: "NJTRST/SPI1_MISO/USART1_CTS_NSS"
- note added: "OCTOSPI_CLK/SPI2_SCK/TIM2_CH3/USART3_TX"
- note added: "OCTOSPI_CLK/TIM2_CH4/USART2_RX"
- note added: "OCTOSPI_DQS"
- note added: "OCTOSPI_DQS/I2C1_SMBA/SPI1_SCK/TIM2_CH2/USART2_RTS_DE"
- note added: "OCTOSPI_IO0/TIM1_CH3N/USART3_RTS_DE"
- note added: "OCTOSPI_IO1/TIM1_CH2N/SPI1_NSS/USART3_CK"
- note added: "OCTOSPI_IO2/TIM1_CH1N/SPI1_MOSI"
- note added: "OCTOSPI_IO3/TIM1_BKIN/SPI1_MISO/USART3_CTS_NSS"
- note added: "OCTOSPI_IO4/SPI2_MOSI"
- note added: "OCTOSPI_IO5/SPI2_MISO"
- note added: "OCTOSPI_IO6/SPI2_MOSI"
- note added: "OCTOSPI_IO7"
- note added: "OCTOSPI_IO7/USART3_TX"
- note added: "OCTOSPI_NCLK/I2C1_SMBA/SPI1_MOSI/USART1_CK"
- note added: "OCTOSPI_NCLK/TIM1_BKIN/SPI2_NSS/USART3_CK"
- note added: "OCTOSPI_NCS/SPI1_NSS/USART2_CK"
- note added: "OCTOSPI_NCS/TIM2_CH3/USART2_TX"
- note added: "OCTOSPI_NCS/TIM2_CH4/USART3_RX"
- note added: "OCTOSPI_NCS/USART3_RX/USART4_RX"
- note added: "SPI1_SCK/TIM2_CH1/TIM2_ETR"
- note added: "TIM1_CH1/USART1_CK"
- note added: "TIM1_CH1N/SPI2_SCK/USART3_CTS_NSS"
- note added: "TIM1_CH2/SPI2_SCK/USART1_TX"
- note added: "TIM1_CH2N/SPI2_MISO/USART3_RTS_DE"
- note added: "TIM1_CH3/USART1_RX"
- note added: "TIM1_CH3N/SPI2_MOSI/USB_CC2"
- note added: "TIM1_CH4/TIM1_BKIN2/SPI1_MISO/USB_DM/USART1_CTS_NSS"
- note added: "TIM1_ETR/SPI1_MOSI/USB_DP/USART1_RTS_DE"
- note added: "TIM2_CH1/TIM2_ETR/USART2_CTS_NSS"
- note added: "USART3_CK"
- note added: "USART3_RTS_DE"
- note added: "USART3_RX"
- note added: "USART3_TX/USART4_TX"
- note added: "USB_NOE"
- note added: "Verified"
- note removed: "1.8 V"
- note removed: "3.0 V"
- note removed: "COLMUX_D = 0 -> Cols 0-7 COLMUX_D = 1 -> Cols 8-14"
- note removed: "Via to GND-layer on PVSS1"
- note removed: "Via to GND-layer on PVSS2"

Commit message: Lotta Changes, Initial Routing
Parts:
- removed D10, D108, D11, D110, D12, D121, D127, D128, D129, D13, D130, D132, D137, D14, D142, D147, D15, D152, D157, D16, D162, D167, D17, D172, D177, D18, D182, D187, D19, D20, D21, D22, D23, D24, D25, D26, D27, D28, D29, D30, D31, D32, D33, D34, D35, D36, D37, D38, D39, D40, D41, D42, D43, D44, D45, D46, D47, D48, D49, D50, D51, D52, D53, D54, D55, D58, D62, D63, D64, D65: WS2812B, LED_SMD:LED_WS2812B_PLCC4_5.0x5.0mm_P3.2mm, symbol LED:WS2812B
- removed D2: LED, LED_SMD:LED_0603_1608Metric_Pad1.05x0.95mm_HandSolder, symbol Device:LED
- removed D56, D57, D59, D60, D61: D, Diode_SMD:D_SOD-123, symbol Device:D
- removed K10: KEYSW, MX_Hotswap:MX-Hotswap-2.25U, symbol keyboard_parts:KEYSW
- removed K11, K12: KEYSW, MX_Hotswap:MX-Hotswap-1.25U, symbol keyboard_parts:KEYSW
- removed K8, K9: KEYSW, MX_Hotswap:MX-Hotswap-1.5U, symbol keyboard_parts:KEYSW
- removed R3: 10k, Resistor_SMD:R_0402_1005Metric, symbol Device:R
- removed TP1: VBAT, TestPoint:TestPoint_Pad_2.5x2.5mm, symbol Connector:TestPoint
- removed TP2: Switch_OUT, TestPoint:TestPoint_Pad_2.5x2.5mm, symbol Connector:TestPoint
- removed TP3: IN1, TestPoint:TestPoint_Pad_2.5x2.5mm, symbol Connector:TestPoint
- added C10, C12, C8, C9: 100nF, Capacitor_SMD:C_0603_1608Metric_Pad1.08x0.95mm_HandSolder, symbol Device:C
- added C13, C15: 1uF, Capacitor_SMD:C_0603_1608Metric_Pad1.08x0.95mm_HandSolder, symbol Device:C
- added C14: 4.7uF, Capacitor_SMD:C_0603_1608Metric_Pad1.08x0.95mm_HandSolder, symbol Device:C
- added C16, C17: 10nF, Capacitor_SMD:C_0603_1608Metric_Pad1.08x0.95mm_HandSolder, symbol Device:C
- added C5, C7: C, Capacitor_SMD:C_0603_1608Metric_Pad1.08x0.95mm_HandSolder, symbol Device:C
- added D141: LED, LED_SMD:LED_0603_1608Metric_Pad1.05x0.95mm_HandSolder, symbol Device:LED
- added LED1, LED10, LED11, LED12, LED13, LED14, LED16, LED17, LED18, LED19, LED2, LED20, LED21, LED22, LED23, LED24, LED25, LED26, LED27, LED28, LED29, LED3, LED31, LED32, LED33, LED34, LED35, LED36, LED37, LED38, LED39, LED4, LED40, LED41, LED42, LED43, LED44, LED46, LED47, LED48, LED49, LED5, LED50, LED51, LED52, LED53, LED54, LED55, LED56, LED57, LED58, LED59, LED6, LED61, LED62, LED63, LED64, LED65, LED66, LED67, LED68, LED69, LED7, LED8, LED9: WS2812B, Keebio-Parts.pretty-master:SK6812-MINI-E, symbol LED:WS2812B
- added Y1: Crystal, LIB_NX5032GA-16.000M-LN-CD-1:NX5032GA16000000MHZLNCD1, symbol Device:Crystal
- IC1: footprint SOP65P640X120-16N -> SN74HC251PWR:SOP65P640X120-16N
- IC2, IC3: footprint SOP65P640X120-16N -> SN74LV138APWR:SOP65P640X120-16N
- IC4: footprint BluetoothModuleLibrary:BGM220PC22HNA2R -> (none)
- IC5: footprint SwitchingICLibrary:SON65P300X300X100-9N-D -> LIB_TPS2113ADRBR:SON65P300X300X100-9N-D
- J1: footprint Connector_USB:USB_C_Receptacle_GCT_USB4135-GF-A_6P_TopMnt_Horizontal -> Connector_USB:USB_C_Receptacle_GCT_USB4105-xx-A_16P_TopMnt_Horizontal
- K14: renamed from K3; footprint MX_Hotswap:MX-Hotswap-1.5U -> MX_Hotswap:MX-Hotswap-2U
- K44: renamed from K123; footprint MX_Hotswap:MX-Hotswap-2.25U -> MX_Hotswap:MX-Hotswap-1U
- K47: renamed from K4; footprint MX_Hotswap:MX-Hotswap-2.25U -> MX_Hotswap:MX-Hotswap-1U
- K57: renamed from K115; footprint MX_Hotswap:MX-Hotswap-1U -> MX_Hotswap:MX-Hotswap-2.75U
- K58: renamed from K6; footprint MX_Hotswap:MX-Hotswap-2.25U -> MX_Hotswap:MX-Hotswap-1U
- K59: renamed from K124; footprint MX_Hotswap:MX-Hotswap-1.25U -> MX_Hotswap:MX-Hotswap-1U
- K65: renamed from K7; footprint MX_Hotswap:MX-Hotswap-2.25U -> MX_Hotswap:MX-Hotswap-1.25U
- K69: renamed from K2; footprint MX_Hotswap:MX-Hotswap-1.25U -> MX_Hotswap:MX-Hotswap-1U
- R1, R2, R4, R5, R6: footprint Resistor_SMD:R_0402_1005Metric -> Resistor_SMD:R_0603_1608Metric_Pad0.98x0.95mm_HandSolder
- U4: footprint SOC008_SPA -> S25FL127SABMFI101:SOC008_SPA
- renumbered D104 to D10, D109 to D11, D114 to D12, D119 to D13, D123 to D14, D66 to D16, D71 to D17, D75 to D18, D80 to D19, D70 to D2, D84 to D20, D88 to D21, D93 to D22, D97 to D23, D101 to D24, D105 to D25, D5 to D26, D115 to D27, D120 to D28, D124 to D29, D74 to D3, D67 to D31, D72 to D32, D76 to D33, D81 to D34, D85 to D35, D89 to D36, D94 to D37, D98 to D38, D102 to D39, D79 to D4, D106 to D40, D111 to D41, D116 to D42, D7 to D43, D125 to D44, D68 to D46, D6 to D47, D77 to D48, D82 to D49, D83 to D5, D86 to D50, D90 to D51, D95 to D52, D99 to D53, D103 to D54, D107 to D55, D112 to D56, D117 to D57, D8 to D58, D126 to D59, D87 to D6, D69 to D61, D73 to D62, D78 to D63, D91 to D64, D9 to D65, D113 to D66, D118 to D67, D122 to D68, D4 to D69, D92 to D7, D96 to D8, D100 to D9, K01 to K1, K102 to K10, K107 to K11, K112 to K12, K117 to K13, K64 to K16, K69 to K17, K73 to K18, K78 to K19, K68 to K2, K82 to K20, K86 to K21, K91 to K22, K95 to K23, K99 to K24, K103 to K25, K108 to K26, K113 to K27, K118 to K28, K122 to K29, K72 to K3, K65 to K31, K70 to K32, K74 to K33, K79 to K34, K83 to K35, K87 to K36, K92 to K37, K96 to K38, K100 to K39, K77 to K4, K104 to K40, K109 to K41, K114 to K42, K5 to K43, K66 to K46, K75 to K48, K80 to K49, K81 to K5, K84 to K50, K88 to K51, K93 to K52, K97 to K53, K101 to K54, K105 to K55, K110 to K56, K85 to K6, K67 to K61, K71 to K62, K76 to K63, K89 to K64, K111 to K66, K116 to K67, K120 to K68, K90 to K7, K94 to K8, K98 to K9
Connections:
- net 3V3: now also U3.1 (VBAT), U3.13 (VDDA), U3.19 (VDD), U3.32 (VDD), U3.48 (VDDUSB), U3.64 (VDD), C10.2, C12.2, C13.2, C14.2, C15.2, C16.2, C17.2, C8.2, C9.2
- net COLMUX_A: no longer U3.10 (PC2)
- net COLMUX_B: no longer U3.11 (PC3)
- net COLMUX_C: no longer U3.24 (PC4)
- net COLMUX_OUTA: no longer U3.8 (PC0)
- net COLMUX_OUTB: no longer U3.9 (PC1)
- net EM4_WAKEUP: no longer U3.21 (PA5), U3.56 (PB4)
- net GND: now also U3.60 (PH3), C10.1, C12.1, C13.1, C14.1, C15.1, C16.1, C17.1, C5.2, C7.2, C8.1, C9.1, D141.1 (K), LED1.3 (VSS), LED10.3 (VSS), LED11.3 (VSS), LED12.3 (VSS), LED13.3 (VSS), LED14.3 (VSS), LED16.3 (VSS), LED17.3 (VSS), LED18.3 (VSS), LED19.3 (VSS), LED2.3 (VSS), LED20.3 (VSS), LED21.3 (VSS), LED22.3 (VSS), LED23.3 (VSS), LED24.3 (VSS), LED25.3 (VSS), LED26.3 (VSS), LED27.3 (VSS), LED28.3 (VSS), LED29.3 (VSS), LED3.3 (VSS), LED31.3 (VSS), LED32.3 (VSS), LED33.3 (VSS), LED34.3 (VSS), LED35.3 (VSS), LED36.3 (VSS), LED37.3 (VSS), LED38.3 (VSS), LED39.3 (VSS), LED4.3 (VSS), LED40.3 (VSS), LED41.3 (VSS), LED42.3 (VSS), LED43.3 (VSS), LED44.3 (VSS), LED46.3 (VSS), LED47.3 (VSS), LED48.3 (VSS), LED49.3 (VSS), LED5.3 (VSS), LED50.3 (VSS), LED51.3 (VSS), LED52.3 (VSS), LED53.3 (VSS), LED54.3 (VSS), LED55.3 (VSS), LED56.3 (VSS), LED57.3 (VSS), LED58.3 (VSS), LED59.3 (VSS), LED6.3 (VSS), LED61.3 (VSS), LED62.3 (VSS), LED63.3 (VSS), LED64.3 (VSS), LED65.3 (VSS), LED66.3 (VSS), LED67.3 (VSS), LED68.3 (VSS), LED69.3 (VSS), LED7.3 (VSS), LED8.3 (VSS), LED9.3 (VSS)
- net ROW0_LED: now also LED1.4 (DIN)
- net ROW1_LED: now also LED16.4 (DIN)
- net ROW2_LED: now also LED31.4 (DIN)
- net ROW3_LED: now also LED46.4 (DIN)
- net ROW4_LED: now also LED61.4 (DIN)
- net ROWDEMUX_A: no longer U3.25 (PC5)
- net ROWDEMUX_B: no longer U3.37 (PC6)
- net ROWDEMUX_C: no longer U3.38 (PC7)
- net Switch_OUT: now also LED1.1 (VDD), LED10.1 (VDD), LED11.1 (VDD), LED12.1 (VDD), LED13.1 (VDD), LED14.1 (VDD), LED16.1 (VDD), LED17.1 (VDD), LED18.1 (VDD), LED19.1 (VDD), LED2.1 (VDD), LED20.1 (VDD), LED21.1 (VDD), LED22.1 (VDD), LED23.1 (VDD), LED24.1 (VDD), LED25.1 (VDD), LED26.1 (VDD), LED27.1 (VDD), LED28.1 (VDD), LED29.1 (VDD), LED3.1 (VDD), LED31.1 (VDD), LED32.1 (VDD), LED33.1 (VDD), LED34.1 (VDD), LED35.1 (VDD), LED36.1 (VDD), LED37.1 (VDD), LED38.1 (VDD), LED39.1 (VDD), LED4.1 (VDD), LED40.1 (VDD), LED41.1 (VDD), LED42.1 (VDD), LED43.1 (VDD), LED44.1 (VDD), LED46.1 (VDD), LED47.1 (VDD), LED48.1 (VDD), LED49.1 (VDD), LED5.1 (VDD), LED50.1 (VDD), LED51.1 (VDD), LED52.1 (VDD), LED53.1 (VDD), LED54.1 (VDD), LED55.1 (VDD), LED56.1 (VDD), LED57.1 (VDD), LED58.1 (VDD), LED59.1 (VDD), LED6.1 (VDD), LED61.1 (VDD), LED62.1 (VDD), LED63.1 (VDD), LED64.1 (VDD), LED65.1 (VDD), LED66.1 (VDD), LED67.1 (VDD), LED68.1 (VDD), LED69.1 (VDD), LED7.1 (VDD), LED8.1 (VDD), LED9.1 (VDD)
- net at U3.5 (PH0): now also C5.1, Y1.1
- net at U3.6 (PH1): now also C7.1, Y1.2
- net at R6.2: now also D141.2 (A)
- net CC1: no longer names the net of J1.A5 (CC1)
- net CC2: no longer names the net of J1.B5 (CC2)
- net ~{BLUETOOTH_LED} renamed BLUETOOTH_STATUS
- new net: LED34.2 (DOUT), LED35.4 (DIN)
- new net: LED33.2 (DOUT), LED34.4 (DIN)
- new net: LED66.2 (DOUT), LED67.4 (DIN)
- new net: LED65.2 (DOUT), LED66.4 (DIN)
- new net: LED10.2 (DOUT), LED11.4 (DIN)
- new net: LED10.4 (DIN), LED9.2 (DOUT)
- new net: LED47.2 (DOUT), LED48.4 (DIN)
- new net: LED46.2 (DOUT), LED47.4 (DIN)
- new net: LED17.2 (DOUT), LED18.4 (DIN)
- new net: LED16.2 (DOUT), LED17.4 (DIN)
- new net: LED43.2 (DOUT), LED44.4 (DIN)
- new net: LED5.2 (DOUT), LED6.4 (DIN)
- new net: LED4.2 (DOUT), LED5.4 (DIN)
- new net: LED37.2 (DOUT), LED38.4 (DIN)
- new net: LED36.2 (DOUT), LED37.4 (DIN)
- new net: LED63.2 (DOUT), LED64.4 (DIN)
- new net: LED62.2 (DOUT), LED63.4 (DIN)
- new net: LED41.2 (DOUT), LED42.4 (DIN)
- new net: LED40.2 (DOUT), LED41.4 (DIN)
- new net: LED31.2 (DOUT), LED32.4 (DIN)
- new net: LED32.2 (DOUT), LED33.4 (DIN)
- new net: LED55.2 (DOUT), LED56.4 (DIN)
- new net: LED54.2 (DOUT), LED55.4 (DIN)
- new net: LED58.2 (DOUT), LED59.4 (DIN)
- new net: LED35.2 (DOUT), LED36.4 (DIN)
- new net: LED19.2 (DOUT), LED20.4 (DIN)
- new net: LED18.2 (DOUT), LED19.4 (DIN)
- new net: LED21.2 (DOUT), LED22.4 (DIN)
- new net: LED20.2 (DOUT), LED21.4 (DIN)
- new net: LED39.2 (DOUT), LED40.4 (DIN)
- new net: LED38.2 (DOUT), LED39.4 (DIN)
- new net: LED28.2 (DOUT), LED29.4 (DIN)
- new net: LED27.2 (DOUT), LED28.4 (DIN)
- new net: LED3.2 (DOUT), LED4.4 (DIN)
- new net: LED2.2 (DOUT), LED3.4 (DIN)
- new net: LED1.2 (DOUT), LED2.4 (DIN)
- new net: LED42.2 (DOUT), LED43.4 (DIN)
- new net: LED23.2 (DOUT), LED24.4 (DIN)
- new net: LED22.2 (DOUT), LED23.4 (DIN)
- new net: LED8.2 (DOUT), LED9.4 (DIN)
- new net: LED7.2 (DOUT), LED8.4 (DIN)
- new net: LED61.2 (DOUT), LED62.4 (DIN)
- new net: LED12.2 (DOUT), LED13.4 (DIN)
- new net: LED11.2 (DOUT), LED12.4 (DIN)
- new net: LED48.2 (DOUT), LED49.4 (DIN)
- new net: LED26.2 (DOUT), LED27.4 (DIN)
- new net: LED6.2 (DOUT), LED7.4 (DIN)
- new net: LED56.2 (DOUT), LED57.4 (DIN)
- new net: LED51.2 (DOUT), LED52.4 (DIN)
- new net: LED50.2 (DOUT), LED51.4 (DIN)
- new net: LED67.2 (DOUT), LED68.4 (DIN)
- new net: LED13.2 (DOUT), LED14.4 (DIN)
- new net: LED68.2 (DOUT), LED69.4 (DIN)
- new net: LED57.2 (DOUT), LED58.4 (DIN)
- new net: LED64.2 (DOUT), LED65.4 (DIN)
- new net: LED53.2 (DOUT), LED54.4 (DIN)
- new net: LED49.2 (DOUT), LED50.4 (DIN)
- new net: LED52.2 (DOUT), LED53.4 (DIN)
- new net: LED25.2 (DOUT), LED26.4 (DIN)
- new net: LED24.2 (DOUT), LED25.4 (DIN)
- no-connect marks 34 -> 29
Other:
- note added: "safely un jtagged"
- note removed: "MACRO1"
- note removed: "MACRO2"
- note removed: "MACRO3"
- note removed: "MACRO4"
- note removed: "MACRO5"
- moved on the sheet: SW1, U2, U3

Commit message: I am very good at using version control, BIG UPDATE see desc
This commit contains version 1 of the daughterboard prototype for the key switch and SK6812-E LED matrix and it already contains a mistake with the floating G2 pin on the row demux :)
Parts:
- removed BT1, BT2, BT3: 1.5V, symbol BA1AAPC:BA1AAPC
- removed C10, C12, C8, C9: 100nF, Capacitor_SMD:C_0603_1608Metric_Pad1.08x0.95mm_HandSolder, symbol Device:C
- removed C11: 4.7uF, Capacitor_SMD:C_0603_1608Metric_Pad1.08x0.95mm_HandSolder, symbol Device:C_Polarized_Small_US
- removed C13, C15: 1uF, Capacitor_SMD:C_0603_1608Metric_Pad1.08x0.95mm_HandSolder, symbol Device:C
- removed C14: 4.7uF, Capacitor_SMD:C_0603_1608Metric_Pad1.08x0.95mm_HandSolder, symbol Device:C
- removed C16, C17: 10nF, Capacitor_SMD:C_0603_1608Metric_Pad1.08x0.95mm_HandSolder, symbol Device:C
- removed C3: 1.0u, Capacitor_SMD:C_0603_1608Metric_Pad1.08x0.95mm_HandSolder, symbol Device:C
- removed C4: 0.01u, Capacitor_SMD:C_0603_1608Metric_Pad1.08x0.95mm_HandSolder, symbol Device:C
- removed C5, C7: C, Capacitor_SMD:C_0603_1608Metric_Pad1.08x0.95mm_HandSolder, symbol Device:C
- removed C6: 0.1uF, Capacitor_SMD:C_0603_1608Metric_Pad1.08x0.95mm_HandSolder, symbol Device:C_Small
- removed D141: LED, LED_SMD:LED_0603_1608Metric_Pad1.05x0.95mm_HandSolder, symbol Device:LED
- removed IC4: BGM220PC22HNA2R, symbol BGM220PC22HNA2R:BGM220PC22HNA2R
- removed IC5: TPS2113ADRBR, LIB_TPS2113ADRBR:SON65P300X300X100-9N-D, symbol TPS2113ADRBR:TPS2113ADRBR
- removed J1: USB_C_Receptacle_USB2.0, Connector_USB:USB_C_Receptacle_GCT_USB4105-xx-A_16P_TopMnt_Horizontal, symbol Connector:USB_C_Receptacle_USB2.0
- removed J2: Conn_ARM_JTAG_SWD_10, Connector_PinHeader_2.54mm:PinHeader_2x05_P2.54mm_Vertical, symbol Connector:Conn_ARM_JTAG_SWD_10
- removed J3: Conn_02x05_Odd_Even, Connector_PinHeader_1.27mm:PinHeader_2x05_P1.27mm_Vertical, symbol Connector_Generic:Conn_02x05_Odd_Even
- removed J4: BATT_POS, Connector_Pin:Pin_D1.0mm_L10.0mm, symbol Connector:Conn_01x01_Pin
- removed J5: BATT_NEG, Connector_Pin:Pin_D1.0mm_L10.0mm, symbol Connector:Conn_01x01_Pin
- removed R1, R4: 22, Resistor_SMD:R_0603_1608Metric_Pad0.98x0.95mm_HandSolder, symbol Device:R
- removed R2: 10k, Resistor_SMD:R_0603_1608Metric_Pad0.98x0.95mm_HandSolder, symbol Device:R
- removed R5: 750, Resistor_SMD:R_0603_1608Metric_Pad0.98x0.95mm_HandSolder, symbol Device:R
- removed R6: 1.1k, Resistor_SMD:R_0603_1608Metric_Pad0.98x0.95mm_HandSolder, symbol Device:R
- removed SW1: RotaryEncoder_Switch, symbol Device:RotaryEncoder_Switch
- removed SW2: BAT_SWITCH, SLW-121586-5A-D:SLW1215865AD, symbol Switch:SW_SPDT
- removed TP4: 3V3, TestPoint:TestPoint_Pad_2.5x2.5mm, symbol Connector:TestPoint
- removed U1: Adafruit ST7735R, footprints:adafruit_st7735r, symbol adafruit_st7735r:Adafruit ST7735R
- removed U2: VEML6030, VEML6030:Vishay-6.550-5348.01-4-02_2016-1-MFG, symbol eec:VEML6030
- removed U3: STM32L552RETx, Package_QFP:LQFP-64_10x10mm_P0.5mm, symbol MCU_ST_STM32L5:STM32L552RETx
- removed U4: S25FL127SABMFI101, S25FL127SABMFI101:SOC008_SPA, symbol 2023-12-04_00-10-28:S25FL127SABMFI101
- removed U5: TPS73633DBV, Package_TO_SOT_SMD:SOT-23-5, symbol Regulator_Linear:TPS73633DBV
- removed Y1: Crystal, LIB_NX5032GA-16.000M-LN-CD-1:NX5032GA16000000MHZLNCD1, symbol Device:Crystal
- added JP1, JP2, JP3, JP4, JP5, JP6: SolderJumper_2_Bridged, Jumper:SolderJumper-2_P1.3mm_Bridged_RoundedPad1.0x1.5mm, symbol Jumper:SolderJumper_2_Bridged
- added U1: TXB0108DQSR, Package_SON:USON-20_2x4mm_P0.4mm, symbol Logic_LevelTranslator:TXB0108DQSR
- added U6: STM32L552ZETxQ, STZio:STZio, symbol STZio:STM32L552ZETxQ_Zio
- C1, C2: value 0.1u -> 0.1uF
Connections:
- net COL14 is gone; now on net COL13: IC3.13 (D6)
- net ROW1_LED is gone; now on an unnamed net: LED16.4 (DIN)
- net ROW2_LED is gone; now on an unnamed net: LED31.4 (DIN)
- net ROW3_LED is gone; now on an unnamed net: LED46.4 (DIN)
- net VBAT is gone; now on net GND: C1.1
- net VBUS is gone; now on net GND: C2.1
- net 3V3: now also C1.2, U1.5 (VCCA), U6.7 (3V3)
- net COL1: now also IC3.4 (D0); no longer IC1.3 (D1)
- net COL10: now also IC1.14 (D5); no longer IC3.2 (D2)
- net COL11: now also IC3.14 (D5); no longer IC3.1 (D3)
- net COL12: now also IC1.13 (D6); no longer IC3.15 (D4)
- net COL13: no longer IC3.14 (D5)
- net COL2: now also IC1.3 (D1); no longer IC1.2 (D2)
- net COL3: now also IC3.3 (D1); no longer IC1.1 (D3)
- net COL4: now also IC1.2 (D2); no longer IC1.15 (D4)
- net COL5: now also IC3.2 (D2); no longer IC1.14 (D5)
- net COL6: now also IC1.1 (D3); no longer IC1.13 (D6)
- net COL7: now also IC3.1 (D3); no longer IC1.12 (D7)
- net COL8: now also IC1.15 (D4); no longer IC3.4 (D0)
- net COL9: now also IC3.15 (D4); no longer IC3.3 (D1)
- net COLMUX_A: now also U6.34 (PE5)
- net COLMUX_B: now also U6.36 (PE6)
- net COLMUX_C: now also U6.38 (PE3)
- net COLMUX_OUTA: now also U6.16 (PF5)
- net COLMUX_OUTB: now also U6.46 (PG1)
- net GND: now also U1.15 (GND), U6.11 (GND), U6.13 (GND), U6.28 (GND), U6.39 (GND), U6.54 (GND), U6.67 (AVDD), U6.69 (AGND), U6.71 (GND), U6.83 (GND), U6.88 (GND), U6.93 (GND); no longer C1.2, C2.2
- net ROWDEMUX_A: now also U6.27 (PC0)
- net ROWDEMUX_B: now also U6.32 (PE4)
- net ROWDEMUX_C: now also U6.30 (PE2)
- net at LED34.2 (DOUT): now also LED33.4 (DIN); no longer LED35.4 (DIN)
- net at LED34.4 (DIN): now also LED35.2 (DOUT); no longer LED33.2 (DOUT)
- net at LED66.2 (DOUT): now also LED65.4 (DIN); no longer LED67.4 (DIN)
- net at LED66.4 (DIN): now also LED67.2 (DOUT); no longer LED65.2 (DOUT)
- net at LED10.2 (DOUT): now also LED9.4 (DIN); no longer LED11.4 (DIN)
- net at LED10.4 (DIN): now also LED11.2 (DOUT); no longer LED9.2 (DOUT)
- net at LED47.2 (DOUT): no longer LED48.4 (DIN)
- net at LED47.4 (DIN): now also LED48.2 (DOUT); no longer LED46.2 (DOUT)
- net at LED17.2 (DOUT): no longer LED18.4 (DIN)
- net at LED17.4 (DIN): now also LED18.2 (DOUT); no longer LED16.2 (DOUT)
- net at LED44.2 (DOUT): now also LED43.4 (DIN)
- net at LED43.2 (DOUT): now also LED42.4 (DIN); no longer LED44.4 (DIN)
- net at LED5.2 (DOUT): now also LED4.4 (DIN); no longer LED6.4 (DIN)
- net at LED5.4 (DIN): now also LED6.2 (DOUT); no longer LED4.2 (DOUT)
- net at LED37.2 (DOUT): now also LED36.4 (DIN); no longer LED38.4 (DIN)
- net at LED37.4 (DIN): now also LED38.2 (DOUT); no longer LED36.2 (DOUT)
- net at LED63.2 (DOUT): now also LED62.4 (DIN); no longer LED64.4 (DIN)
- net at LED63.4 (DIN): now also LED64.2 (DOUT); no longer LED62.2 (DOUT)
- net at LED41.2 (DOUT): now also LED40.4 (DIN); no longer LED42.4 (DIN)
- net at LED41.4 (DIN): now also LED42.2 (DOUT); no longer LED40.2 (DOUT)
- net at LED31.2 (DOUT): no longer LED32.4 (DIN)
- net at LED32.2 (DOUT): no longer LED33.4 (DIN)
- net at LED55.2 (DOUT): now also LED54.4 (DIN); no longer LED56.4 (DIN)
- net at LED55.4 (DIN): now also LED56.2 (DOUT); no longer LED54.2 (DOUT)
- net at LED59.2 (DOUT): now also LED58.4 (DIN)
- net at LED58.2 (DOUT): now also LED57.4 (DIN); no longer LED59.4 (DIN)
- net at LED19.2 (DOUT): now also LED18.4 (DIN); no longer LED20.4 (DIN)
- net at LED19.4 (DIN): now also LED20.2 (DOUT); no longer LED18.2 (DOUT)
- net at LED21.2 (DOUT): now also LED20.4 (DIN); no longer LED22.4 (DIN)
- net at LED21.4 (DIN): now also LED22.2 (DOUT); no longer LED20.2 (DOUT)
- net at LED39.2 (DOUT): now also LED38.4 (DIN); no longer LED40.4 (DIN)
- net at LED39.4 (DIN): now also LED40.2 (DOUT); no longer LED38.2 (DOUT)
- net at LED28.2 (DOUT): now also LED27.4 (DIN); no longer LED29.4 (DIN)
- net at LED28.4 (DIN): now also LED29.2 (DOUT); no longer LED27.2 (DOUT)
- net at LED3.2 (DOUT): now also LED2.4 (DIN); no longer LED4.4 (DIN)
- net at LED3.4 (DIN): now also LED4.2 (DOUT); no longer LED2.2 (DOUT)
- net at LED1.2 (DOUT): no longer LED2.4 (DIN)
- net at LED23.2 (DOUT): now also LED22.4 (DIN); no longer LED24.4 (DIN)
- net at LED23.4 (DIN): now also LED24.2 (DOUT); no longer LED22.2 (DOUT)
- net at LED8.2 (DOUT): now also LED7.4 (DIN); no longer LED9.4 (DIN)
- net at LED8.4 (DIN): now also LED9.2 (DOUT); no longer LED7.2 (DOUT)
- net at LED61.2 (DOUT): no longer LED62.4 (DIN)
- net at LED12.2 (DOUT): now also LED11.4 (DIN); no longer LED13.4 (DIN)
- net at LED12.4 (DIN): now also LED13.2 (DOUT); no longer LED11.2 (DOUT)
- net at LED49.4 (DIN): now also LED50.2 (DOUT); no longer LED48.2 (DOUT)
- net at LED26.2 (DOUT): now also LED25.4 (DIN); no longer LED27.4 (DIN)
- net at LED51.2 (DOUT): now also LED50.4 (DIN); no longer LED52.4 (DIN)
- net at LED51.4 (DIN): now also LED52.2 (DOUT); no longer LED50.2 (DOUT)
- net at LED68.4 (DIN): now also LED69.2 (DOUT); no longer LED67.2 (DOUT)
- net ROW0_LED_5V: now reaches LED14.4 (DIN)
- net ROW0_LED_5V: now also U1.20 (B1); no longer LED13.2 (DOUT)
- net at LED68.2 (DOUT): now also LED67.4 (DIN); no longer LED69.4 (DIN)
- net at LED57.2 (DOUT): now also LED56.4 (DIN); no longer LED58.4 (DIN)
- net at LED53.2 (DOUT): now also LED52.4 (DIN); no longer LED54.4 (DIN)
- net at LED49.2 (DOUT): now also LED48.4 (DIN); no longer LED50.4 (DIN)
- net at LED14.2 (DOUT): now also LED13.4 (DIN)
- net at LED53.4 (DIN): now also LED54.2 (DOUT); no longer LED52.2 (DOUT)
- net at LED26.4 (DIN): now also LED27.2 (DOUT); no longer LED25.2 (DOUT)
- net ROW0_LED: no longer names the net of LED1.4 (DIN)
- net ROW0_LED: now also LED2.2 (DOUT)
- net ROW4_LED: no longer names the net of LED61.4 (DIN)
- net ROW4_LED: now also LED62.2 (DOUT)
- removed net Switch_OUT: LED1.1 (VDD), LED10.1 (VDD), LED11.1 (VDD), LED12.1 (VDD), LED13.1 (VDD), LED14.1 (VDD), LED16.1 (VDD), LED17.1 (VDD), LED18.1 (VDD), LED19.1 (VDD), LED2.1 (VDD), LED20.1 (VDD), LED21.1 (VDD), LED22.1 (VDD), LED23.1 (VDD), LED24.1 (VDD), LED25.1 (VDD), LED26.1 (VDD), LED27.1 (VDD), LED28.1 (VDD), LED29.1 (VDD), LED3.1 (VDD), LED31.1 (VDD), LED32.1 (VDD), LED33.1 (VDD), LED34.1 (VDD), LED35.1 (VDD), LED36.1 (VDD), LED37.1 (VDD), LED38.1 (VDD), LED39.1 (VDD), LED4.1 (VDD), LED40.1 (VDD), LED41.1 (VDD), LED42.1 (VDD), LED43.1 (VDD), LED44.1 (VDD), LED46.1 (VDD), LED47.1 (VDD), LED48.1 (VDD), LED49.1 (VDD), LED5.1 (VDD), LED50.1 (VDD), LED51.1 (VDD), LED52.1 (VDD), LED53.1 (VDD), LED54.1 (VDD), LED55.1 (VDD), LED56.1 (VDD), LED57.1 (VDD), LED58.1 (VDD), LED59.1 (VDD), LED6.1 (VDD), LED61.1 (VDD), LED62.1 (VDD), LED63.1 (VDD), LED64.1 (VDD), LED65.1 (VDD), LED66.1 (VDD), LED67.1 (VDD), LED68.1 (VDD), LED69.1 (VDD), LED7.1 (VDD), LED8.1 (VDD), LED9.1 (VDD)
- new net: JP4.1 (A), LED31.1 (VDD), LED32.1 (VDD), LED33.1 (VDD), LED34.1 (VDD), LED35.1 (VDD), LED36.1 (VDD), LED37.1 (VDD), LED38.1 (VDD), LED39.1 (VDD), LED40.1 (VDD), LED41.1 (VDD), LED42.1 (VDD), LED43.1 (VDD), LED44.1 (VDD)
- new net: JP5.1 (A), LED46.1 (VDD), LED47.1 (VDD), LED48.1 (VDD), LED49.1 (VDD), LED50.1 (VDD), LED51.1 (VDD), LED52.1 (VDD), LED53.1 (VDD), LED54.1 (VDD), LED55.1 (VDD), LED56.1 (VDD), LED57.1 (VDD), LED58.1 (VDD), LED59.1 (VDD)
- new net: JP6.1 (A), LED61.1 (VDD), LED62.1 (VDD), LED63.1 (VDD), LED64.1 (VDD), LED65.1 (VDD), LED66.1 (VDD), LED67.1 (VDD), LED68.1 (VDD), LED69.1 (VDD)
- new net: JP2.1 (A), LED1.1 (VDD), LED10.1 (VDD), LED11.1 (VDD), LED12.1 (VDD), LED13.1 (VDD), LED14.1 (VDD), LED2.1 (VDD), LED3.1 (VDD), LED4.1 (VDD), LED5.1 (VDD), LED6.1 (VDD), LED7.1 (VDD), LED8.1 (VDD), LED9.1 (VDD)
- new net: JP3.1 (A), LED16.1 (VDD), LED17.1 (VDD), LED18.1 (VDD), LED19.1 (VDD), LED20.1 (VDD), LED21.1 (VDD), LED22.1 (VDD), LED23.1 (VDD), LED24.1 (VDD), LED25.1 (VDD), LED26.1 (VDD), LED27.1 (VDD), LED28.1 (VDD), LED29.1 (VDD)
- new net: C2.2, JP1.1 (A), U1.16 (VCCB)
- new net: LED32.4 (DIN), LED33.2 (DOUT)
- new net: LED35.4 (DIN), LED36.2 (DOUT)
- new net: LED6.4 (DIN), LED7.2 (DOUT)
- new net: LED64.4 (DIN), LED65.2 (DOUT)
- new net: LED24.4 (DIN), LED25.2 (DOUT)
- new net 5V: JP1.2 (B), JP2.2 (B), JP3.2 (B), JP4.2 (B), JP5.2 (B), JP6.2 (B), U6.9 (5V)
- new net LOGIC_TRANS_OE: U1.6 (OE), U6.31 (PB6)
- new net ROW0_LED_3V3: U1.1 (A1), U6.17 (PA3)
- new net ROW1_LED_3V3: U1.2 (A2), U6.19 (PA2)
- new net ROW1_LED_5V: LED29.4 (DIN), U1.19 (B2)
- new net ROW2_LED_3V3: U1.3 (A3), U6.21 (PC3)
- new net ROW2_LED_5V: LED44.4 (DIN), U1.18 (B3)
- new net ROW3_LED_3V3: U1.4 (A4), U6.23 (PB0)
- new net ROW3_LED_5V: LED59.4 (DIN), U1.17 (B4)
- new net ROW4_LED_3V3: U1.7 (A5), U6.25 (PC1)
- new net ROW4_LED_5V: LED69.4 (DIN), U1.14 (B5)
- no-connect marks 29 -> 6
Other:
- note removed: "BLUETOOTH_?X/?TS are relative to the main MCU"
- note removed: "I2C1_SCL"
- note removed: "I2C1_SCL/USART1_TX"
- note removed: "I2C1_SDA/SPI2_NSS"
- note removed: "I2C1_SDA/USART1_RX"
- note removed: "ILIM - Current Limit Current Limit = 500/R TPS2113A can do 630mA min limit R = 500/0.630 ~= 800 Ohm"
- note removed: "JTAG_CLK/SWD_CLK/I2C1_SMBA"
- note removed: "JTAG_TDI/SPI1_NSS/TIM2_CH1/TIM2_ETR/USART2_RX/USART3_RTS_DE/USB_CC1"
- note removed: "JTAG_TDO/SWO/SPI1_SCK/TM2_CH2/USART1_RTS_DE"
- note removed: "JTAG_TMS/SWDIO/USB_NOE"
- note removed: "Must have a large copper ground pour to dissipate heat properly"
- note removed: "NJTRST/SPI1_MISO/USART1_CTS_NSS"
- note removed: "OCTOSPI_CLK/SPI2_SCK/TIM2_CH3/USART3_TX"
- note removed: "OCTOSPI_CLK/TIM2_CH4/USART2_RX"
- note removed: "OCTOSPI_DQS"
- note removed: "OCTOSPI_DQS/I2C1_SMBA/SPI1_SCK/TIM2_CH2/USART2_RTS_DE"
- note removed: "OCTOSPI_IO0/TIM1_CH3N/USART3_RTS_DE"
- note removed: "OCTOSPI_IO1/TIM1_CH2N/SPI1_NSS/USART3_CK"
- note removed: "OCTOSPI_IO2/TIM1_CH1N/SPI1_MOSI"
- note removed: "OCTOSPI_IO3/TIM1_BKIN/SPI1_MISO/USART3_CTS_NSS"
- note removed: "OCTOSPI_IO4/SPI2_MOSI"
- note removed: "OCTOSPI_IO5/SPI2_MISO"
- note removed: "OCTOSPI_IO6/SPI2_MOSI"
- note removed: "OCTOSPI_IO7"
- note removed: "OCTOSPI_IO7/USART3_TX"
- note removed: "OCTOSPI_NCLK/I2C1_SMBA/SPI1_MOSI/USART1_CK"
- note removed: "OCTOSPI_NCLK/TIM1_BKIN/SPI2_NSS/USART3_CK"
- note removed: "OCTOSPI_NCS/SPI1_NSS/USART2_CK"
- note removed: "OCTOSPI_NCS/TIM2_CH3/USART2_TX"
- note removed: "OCTOSPI_NCS/TIM2_CH4/USART3_RX"
- note removed: "OCTOSPI_NCS/USART3_RX/USART4_RX"
- note removed: "SPI1_SCK/TIM2_CH1/TIM2_ETR"
- note removed: "TIM1_CH1/USART1_CK"
- note removed: "TIM1_CH1N/SPI2_SCK/USART3_CTS_NSS"
- note removed: "TIM1_CH2/SPI2_SCK/USART1_TX"
- note removed: "TIM1_CH2N/SPI2_MISO/USART3_RTS_DE"
- note removed: "TIM1_CH3/USART1_RX"
- note removed: "TIM1_CH3N/SPI2_MOSI/USB_CC2"
- note removed: "TIM1_CH4/TIM1_BKIN2/SPI1_MISO/USB_DM/USART1_CTS_NSS"
- note removed: "TIM1_ETR/SPI1_MOSI/USB_DP/USART1_RTS_DE"
- note removed: "TIM2_CH1/TIM2_ETR/USART2_CTS_NSS"
- note removed: "USART3_CK"
- note removed: "USART3_RTS_DE"
- note removed: "USART3_RX"
- note removed: "USART3_TX/USART4_TX"
- note removed: "USB_NOE"
- note removed: "Verified"
- note removed: "safely un jtagged"
- moved on the sheet: IC1, IC2, IC3
