File: hw/PCB/PCB.kicad_sch (KiCad schematic)
At the start: 270 parts, among them IC1 TXU0101DCKR, J1 Conn_01x02, J2 Adafruit TFT, J5 Conn_01x05, K1 KEYSW, K10 KEYSW, K11 KEYSW, K12 KEYSW, K13 KEYSW, K14 KEYSW, K15 KEYSW, K16 KEYSW, K17 KEYSW, K18 KEYSW, K19 KEYSW, K2 KEYSW, K20 KEYSW, K21 KEYSW, K22 KEYSW, K23 KEYSW, K24 KEYSW, K25 KEYSW, K26 KEYSW, K27 KEYSW, K28 KEYSW, K29 KEYSW, K3 KEYSW, K31 KEYSW, K32 KEYSW, K33 KEYSW, K34 KEYSW, K35 KEYSW, K36 KEYSW, K37 KEYSW, K38 KEYSW, K39 KEYSW, K4 KEYSW, K40 KEYSW, K41 KEYSW, K42 KEYSW, K43 KEYSW, K46 KEYSW, K47 KEYSW, K48 KEYSW, K49 KEYSW, K5 KEYSW, K50 KEYSW, K51 KEYSW, K52 KEYSW, K53 KEYSW, K54 KEYSW, K55 KEYSW, K56 KEYSW, K57 KEYSW, K58 KEYSW, K59 KEYSW, K6 KEYSW, K61 KEYSW, K62 KEYSW, K63 KEYSW, K64 KEYSW, K65 KEYSW, K66 KEYSW, K67 KEYSW, K68 KEYSW, K69 KEYSW, K7 KEYSW, K8 KEYSW, K9 KEYSW, SW2 RotaryEncoder_Switch, U1 XIAO-nRF52840-SMD, U3 74HC595, U4 74HC595

Commit message: More routing
Connections:
- net ROW2: now also U1.4 (P0.29_A3_D3); no longer U1.7 (P1.11_D6_TX)
- net ROW3: now also U1.7 (P1.11_D6_TX)
- net ROW4: now also U1.8 (P1.12_D7_RX)
Changed lines of the file:
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@@
+		)
+	)
+	(label "ROW3"
+		(at 49.53 165.1 180)
+		(effects
+			(font
+				(size 1.27 1.27)
+			)
+			(justify right bottom)
 		)
 	)
@@
 		)
 	)
+	(label "ROW4"
+		(at 91.44 165.1 0)
+		(effects
+			(font
+				(size 1.27 1.27)
+			)
+			(justify left bottom)
+		)
+	)
 	(label "TFT_DC"
 		(at 73.66 175.26 270)
@@
 		)
 	)
-	(label "ROW2"
-		(at 49.53 165.1 180)
-		(effects
-			(font
-				(size 1.27 1.27)
-			)
-			(justify right bottom)
-		)
-	)
-	(label "ROW4"
-		(at 96.5646 192.3773 270)
-		(effects
-			(font
-				(size 1.27 1.27)
-			)
-			(justify right bottom)
-		)
-	)
 	(label "COL4"
 		(at 126.365 71.755 0)
@@
 		)
 	)
-	(label "ROW3"
-		(at 88.9 194.31 270)
-		(effects
-			(font
-				(size 1.27 1.27)
-			)
-			(justify right bottom)
-		)
-	)
 	(label "COL_CS"
 		(at 91.44 161.29 0)
@@
 		(effects
 			(font
+				(size 1.27 1.27)
+			)
+			(justify right bottom)
+		)
+	)
+	(label "ROW2"
+		(at 49.53 153.67 180)
+		(effects
+			(font
