File: hw/PCB/PCB.kicad_pcb (KiCad board)
At the start: 2 copper layers, 325 x 95.7 mm, 270 parts, among them IC1 TXU0101DCKR, J1 Conn_01x02, J2 Adafruit TFT, J5 Conn_01x05, K1 KEYSW, K10 KEYSW, K11 KEYSW, K12 KEYSW, K13 KEYSW, K14 KEYSW, K15 KEYSW, K16 KEYSW, K17 KEYSW, K18 KEYSW, K19 KEYSW, K2 KEYSW, K20 KEYSW, K21 KEYSW, K22 KEYSW, K23 KEYSW, K24 KEYSW, K25 KEYSW, K26 KEYSW, K27 KEYSW, K28 KEYSW, K29 KEYSW, K3 KEYSW, K31 KEYSW, K32 KEYSW, K33 KEYSW, K34 KEYSW, K35 KEYSW, K36 KEYSW, K37 KEYSW, K38 KEYSW, K39 KEYSW, K4 KEYSW, K40 KEYSW, K41 KEYSW, K42 KEYSW, K43 KEYSW, K46 KEYSW, K47 KEYSW, K48 KEYSW, K49 KEYSW, K5 KEYSW, K50 KEYSW, K51 KEYSW, K52 KEYSW, K53 KEYSW, K54 KEYSW, K55 KEYSW, K56 KEYSW, K57 KEYSW, K58 KEYSW, K59 KEYSW, K6 KEYSW, K61 KEYSW, K62 KEYSW, K63 KEYSW, K64 KEYSW, K65 KEYSW, K66 KEYSW, K67 KEYSW, K68 KEYSW, K69 KEYSW, K7 KEYSW, K8 KEYSW, K9 KEYSW, SW2 RotaryEncoder_Switch, U1 XIAO-nRF52840-SMD, U3 74HC595, U4 74HC595

Commit message: routing
Parts:
- moved U3 196.8 mm to (318.9, 65.8), turned to 90 degrees
- moved U4 67.1 mm to (327.5, 65.9), turned to 90 degrees
- moved C41 10.7 mm to (32.1, 33.9), turned to 90 degrees
- moved C31 10.5 mm to (222.5, 33.9), turned to 90 degrees
- moved C40 10.5 mm to (51.2, 33.8), turned to 90 degrees
- moved C39 10.5 mm to (70.2, 33.8), turned to 90 degrees
- moved C34 10.4 mm to (165.4, 33.9), turned to 90 degrees
- moved C28 10.4 mm to (289.0, 33.8), turned to 90 degrees
- moved C36 10.4 mm to (127.3, 33.9), turned to 90 degrees
- moved C30 10.4 mm to (241.7, 33.9), turned to 90 degrees
- moved C37 10.4 mm to (108.3, 33.9), turned to 90 degrees
- moved C33 10.4 mm to (184.5, 33.8), turned to 90 degrees
- moved C32 10.4 mm to (203.5, 33.9), turned to 90 degrees
- moved C35 10.4 mm to (146.4, 33.9), turned to 90 degrees
- moved C29 10.3 mm to (260.8, 33.8), turned to 90 degrees
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- renumbered C14 to C11, C15 to C12
Connections:
- LED11 pad 2: Net-(LED11-DOUT) -> Net-(LED10-DIN)
- LED11 pad 4: Net-(LED10-DOUT) -> Net-(LED11-DIN)
- LED12 pad 2: Net-(LED12-DOUT) -> Net-(LED11-DIN)
- LED12 pad 4: Net-(LED11-DOUT) -> Net-(LED12-DIN)
- LED13 pad 2: Net-(LED13-DOUT) -> Net-(LED12-DIN)
- LED13 pad 4: Net-(LED12-DOUT) -> Net-(LED13-DIN)
- LED14 pad 2: unconnected-(LED14-DOUT-Pad2) -> Net-(LED13-DIN)
- LED14 pad 4: Net-(LED13-DOUT) -> Net-(IC1-BY)
- LED16 pad 2: Net-(LED1-DIN) -> Net-(LED16-DOUT)
- LED16 pad 4: Net-(LED16-DIN) -> Net-(LED1-DOUT)
- LED17 pad 2: Net-(LED16-DIN) -> Net-(LED17-DOUT)
- LED17 pad 4: Net-(LED17-DIN) -> Net-(LED16-DOUT)
- LED18 pad 2: Net-(LED17-DIN) -> Net-(LED18-DOUT)
- LED18 pad 4: Net-(LED18-DIN) -> Net-(LED17-DOUT)
- LED19 pad 2: Net-(LED18-DIN) -> Net-(LED19-DOUT)
- LED19 pad 4: Net-(LED19-DIN) -> Net-(LED18-DOUT)
- LED2 pad 2: Net-(LED2-DOUT) -> Net-(LED1-DIN)
- LED2 pad 4: Net-(LED1-DOUT) -> Net-(LED2-DIN)
- LED20 pad 2: Net-(LED19-DIN) -> Net-(LED20-DOUT)
- LED20 pad 4: Net-(LED20-DIN) -> Net-(LED19-DOUT)
- LED21 pad 2: Net-(LED20-DIN) -> Net-(LED21-DOUT)
- LED21 pad 4: Net-(LED21-DIN) -> Net-(LED20-DOUT)
- LED22 pad 2: Net-(LED21-DIN) -> Net-(LED22-DOUT)
- LED22 pad 4: Net-(LED22-DIN) -> Net-(LED21-DOUT)
- LED23 pad 2: Net-(LED22-DIN) -> Net-(LED23-DOUT)
- LED23 pad 4: Net-(LED23-DIN) -> Net-(LED22-DOUT)
- LED24 pad 2: Net-(LED23-DIN) -> Net-(LED24-DOUT)
- LED24 pad 4: Net-(LED24-DIN) -> Net-(LED23-DOUT)
- LED25 pad 2: Net-(LED24-DIN) -> Net-(LED25-DOUT)
- LED25 pad 4: Net-(LED25-DIN) -> Net-(LED24-DOUT)
- LED26 pad 2: Net-(LED25-DIN) -> Net-(LED26-DOUT)
- LED26 pad 4: Net-(LED26-DIN) -> Net-(LED25-DOUT)
- LED27 pad 2: Net-(LED26-DIN) -> Net-(LED27-DOUT)
- LED27 pad 4: Net-(LED27-DIN) -> Net-(LED26-DOUT)
- LED28 pad 2: Net-(LED27-DIN) -> Net-(LED28-DOUT)
- LED28 pad 4: Net-(LED28-DIN) -> Net-(LED27-DOUT)
- LED29 pad 2: Net-(LED28-DIN) -> Net-(LED29-DOUT)
- LED29 pad 4: Net-(LED29-DIN) -> Net-(LED28-DOUT)
- LED3 pad 2: Net-(LED3-DOUT) -> Net-(LED2-DIN)
- LED3 pad 4: Net-(LED2-DOUT) -> Net-(LED3-DIN)
- LED30 pad 2: Net-(LED30-DOUT) -> Net-(LED15-DIN)
- LED30 pad 4: Net-(LED15-DOUT) -> Net-(LED30-DIN)
- LED32 pad 2: Net-(LED32-DOUT) -> Net-(LED31-DIN)
- LED32 pad 4: Net-(LED31-DOUT) -> Net-(LED32-DIN)
- LED33 pad 2: Net-(LED33-DOUT) -> Net-(LED32-DIN)
- LED33 pad 4: Net-(LED32-DOUT) -> Net-(LED33-DIN)
- LED34 pad 2: Net-(LED34-DOUT) -> Net-(LED33-DIN)
- LED34 pad 4: Net-(LED33-DOUT) -> Net-(LED34-DIN)
- LED35 pad 2: Net-(LED35-DOUT) -> Net-(LED34-DIN)
- LED35 pad 4: Net-(LED34-DOUT) -> Net-(LED35-DIN)
- LED36 pad 2: Net-(LED36-DOUT) -> Net-(LED35-DIN)
- LED36 pad 4: Net-(LED35-DOUT) -> Net-(LED36-DIN)
- LED37 pad 2: Net-(LED37-DOUT) -> Net-(LED36-DIN)
- LED37 pad 4: Net-(LED36-DOUT) -> Net-(LED37-DIN)
- LED38 pad 2: Net-(LED38-DOUT) -> Net-(LED37-DIN)
- LED38 pad 4: Net-(LED37-DOUT) -> Net-(LED38-DIN)
- LED39 pad 2: Net-(LED39-DOUT) -> Net-(LED38-DIN)
- LED39 pad 4: Net-(LED38-DOUT) -> Net-(LED39-DIN)
- LED4 pad 2: Net-(LED4-DOUT) -> Net-(LED3-DIN)
- LED4 pad 4: Net-(LED3-DOUT) -> Net-(LED4-DIN)
- LED40 pad 2: Net-(LED40-DOUT) -> Net-(LED39-DIN)
- LED40 pad 4: Net-(LED39-DOUT) -> Net-(LED40-DIN)
- LED41 pad 2: Net-(LED41-DOUT) -> Net-(LED40-DIN)
- LED41 pad 4: Net-(LED40-DOUT) -> Net-(LED41-DIN)
- LED42 pad 2: Net-(LED42-DOUT) -> Net-(LED41-DIN)
- LED42 pad 4: Net-(LED41-DOUT) -> Net-(LED42-DIN)
- LED43 pad 2: Net-(LED29-DIN) -> Net-(LED42-DIN)
- LED43 pad 4: Net-(LED42-DOUT) -> Net-(LED29-DOUT)
- LED46 pad 2: Net-(LED31-DIN) -> Net-(LED46-DOUT)
- LED46 pad 4: Net-(LED46-DIN) -> Net-(LED31-DOUT)
- LED47 pad 2: Net-(LED46-DIN) -> Net-(LED47-DOUT)
- LED47 pad 4: Net-(LED47-DIN) -> Net-(LED46-DOUT)
- LED48 pad 2: Net-(LED47-DIN) -> Net-(LED48-DOUT)
- LED48 pad 4: Net-(LED48-DIN) -> Net-(LED47-DOUT)
- LED49 pad 2: Net-(LED48-DIN) -> Net-(LED49-DOUT)
- LED49 pad 4: Net-(LED49-DIN) -> Net-(LED48-DOUT)
- LED5 pad 2: Net-(LED5-DOUT) -> Net-(LED4-DIN)
- LED5 pad 4: Net-(LED4-DOUT) -> Net-(LED5-DIN)
- LED50 pad 2: Net-(LED49-DIN) -> Net-(LED50-DOUT)
- LED50 pad 4: Net-(LED50-DIN) -> Net-(LED49-DOUT)
- LED51 pad 2: Net-(LED50-DIN) -> Net-(LED51-DOUT)
- LED51 pad 4: Net-(LED51-DIN) -> Net-(LED50-DOUT)
- LED52 pad 2: Net-(LED51-DIN) -> Net-(LED52-DOUT)
- LED52 pad 4: Net-(LED52-DIN) -> Net-(LED51-DOUT)
- LED53 pad 2: Net-(LED52-DIN) -> Net-(LED53-DOUT)
- LED53 pad 4: Net-(LED53-DIN) -> Net-(LED52-DOUT)
- LED54 pad 2: Net-(LED53-DIN) -> Net-(LED54-DOUT)
- LED54 pad 4: Net-(LED54-DIN) -> Net-(LED53-DOUT)
- LED55 pad 2: Net-(LED54-DIN) -> Net-(LED55-DOUT)
- LED55 pad 4: Net-(LED55-DIN) -> Net-(LED54-DOUT)
- LED56 pad 2: Net-(LED55-DIN) -> Net-(LED56-DOUT)
- LED56 pad 4: Net-(LED56-DIN) -> Net-(LED55-DOUT)
- LED57 pad 2: Net-(LED56-DIN) -> Net-(LED57-DOUT)
- LED57 pad 4: Net-(LED57-DIN) -> Net-(LED56-DOUT)
- LED58 pad 2: Net-(LED57-DIN) -> Net-(LED58-DOUT)
- LED58 pad 4: Net-(LED58-DIN) -> Net-(LED57-DOUT)
- LED59 pad 2: Net-(LED58-DIN) -> Net-(LED30-DIN)
- LED59 pad 4: Net-(LED30-DOUT) -> Net-(LED58-DOUT)
- LED6 pad 2: Net-(LED6-DOUT) -> Net-(LED5-DIN)
- LED6 pad 4: Net-(LED5-DOUT) -> Net-(LED6-DIN)
- LED61 pad 2: Net-(LED61-DOUT) -> unconnected-(LED61-DOUT-Pad2)
- LED61 pad 4: Net-(IC1-BY) -> Net-(LED61-DIN)
- LED62 pad 2: Net-(LED62-DOUT) -> Net-(LED61-DIN)
- LED62 pad 4: Net-(LED61-DOUT) -> Net-(LED62-DIN)
- LED63 pad 2: Net-(LED63-DOUT) -> Net-(LED62-DIN)
- LED63 pad 4: Net-(LED62-DOUT) -> Net-(LED63-DIN)
- LED64 pad 2: Net-(LED64-DOUT) -> Net-(LED63-DIN)
- LED64 pad 4: Net-(LED63-DOUT) -> Net-(LED64-DIN)
- LED65 pad 2: Net-(LED65-DOUT) -> Net-(LED64-DIN)
- LED65 pad 4: Net-(LED64-DOUT) -> Net-(LED65-DIN)
- LED66 pad 2: Net-(LED66-DOUT) -> Net-(LED65-DIN)
- LED66 pad 4: Net-(LED65-DOUT) -> Net-(LED66-DIN)
- LED67 pad 2: Net-(LED67-DOUT) -> Net-(LED66-DIN)
- LED67 pad 4: Net-(LED66-DOUT) -> Net-(LED67-DIN)
- LED68 pad 2: Net-(LED15-DIN) -> Net-(LED67-DIN)
- LED68 pad 4: Net-(LED67-DOUT) -> Net-(LED15-DOUT)
- LED7 pad 2: Net-(LED7-DOUT) -> Net-(LED6-DIN)
- LED7 pad 4: Net-(LED6-DOUT) -> Net-(LED7-DIN)
- LED8 pad 2: Net-(LED8-DOUT) -> Net-(LED7-DIN)
- LED8 pad 4: Net-(LED7-DOUT) -> Net-(LED8-DIN)
- LED9 pad 2: Net-(LED10-DIN) -> Net-(LED8-DIN)
- LED9 pad 4: Net-(LED8-DOUT) -> Net-(LED10-DOUT)
- U1 pad 2: /ROW1 -> /ROW0
- U1 pad 3: /ROW0 -> /ROW1
Routing:
- net +5V: track 1387.4 -> 795.7 mm, vias 8 -> 6
- net /ROW2: track 328.5 -> 0.00 mm, vias 16 -> 0
- net /ROW0: track 0.00 -> 301.9 mm, vias 0 -> 1
- net /ROW1: track 0.00 -> 271.4 mm
- net Net-(LED64-DOUT): track 112.9 -> 0.00 mm, vias 8 -> 0
- net Net-(LED64-DIN): track 0.00 -> 112.9 mm, vias 0 -> 8
- net /COL0: track 175.9 -> 76.5 mm, vias 8 -> 5
- net /COL8: track 153.6 -> 76.3 mm, vias 9 -> 6
- net Net-(LED63-DOUT): track 73.5 -> 0.00 mm
- net Net-(LED63-DIN): track 0.00 -> 66.7 mm
- net /COL13: track 174.7 -> 111.9 mm, vias 4 -> 0
- net /COL9: track 142.3 -> 80.4 mm, vias 9 -> 6
- net /COL11: track 118.9 -> 72.9 mm, vias 10 -> 6
- net /COL1: track 135.9 -> 93.8 mm
- net /COL12: track 148.1 -> 112.1 mm, vias 10 -> 8
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Other:
- outline, holes or cut-outs redrawn

Commit message: More routing
Parts:
- moved U3 190.8 mm to (134.2, 113.9), turned to -90 degrees
- moved C10 10.8 mm to (34.4, 110.1), turned to 90 degrees
- moved C7 10.6 mm to (153.5, 110.1), turned to 90 degrees
- moved C60 10.6 mm to (39.2, 72.0), turned to 90 degrees
- moved C2 10.6 mm to (317.8, 110.0), turned to 90 degrees
- moved C6 10.6 mm to (224.9, 110.0), turned to 90 degrees
- moved C54 10.6 mm to (160.6, 71.9), turned to 90 degrees
- moved C56 10.5 mm to (122.5, 72.0), turned to 90 degrees
- moved C49 10.5 mm to (255.9, 72.0), turned to 90 degrees
- moved C4 10.5 mm to (275.0, 110.0), turned to 90 degrees
- moved C48 10.5 mm to (286.8, 72.0), turned to 90 degrees
- moved C3 10.5 mm to (298.8, 110.0), turned to 90 degrees
- moved C8 10.5 mm to (82.0, 110.0), turned to 90 degrees
- moved C50 10.5 mm to (236.8, 72.0), turned to 90 degrees
- moved C52 10.5 mm to (198.7, 72.1), turned to 90 degrees
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Connections:
- U1 pad 4: unconnected-(U1-P0.29_A3_D3-Pad4) -> /ROW2
- U1 pad 7: /ROW2 -> /ROW3
- U1 pad 8: unconnected-(U1-P1.12_D7_RX-Pad8) -> /ROW4
Routing:
- net +5V: track 795.7 -> 1621.4 mm, vias 6 -> 7
- net /ROW4: track 22.4 -> 413.8 mm, vias 4 -> 1
- net /ROW2: track 0.00 -> 331.2 mm, vias 0 -> 1
- net /COL13: track 111.9 -> 21.6 mm
- net Net-(LED63-DIN): track 66.7 -> 0.00 mm
- net Net-(LED64-DIN): track 112.9 -> 66.6 mm, vias 8 -> 0
- net /ROW3: track 318.2 -> 360.4 mm, vias 12 -> 1
- net /COL12: track 112.1 -> 71.1 mm, vias 8 -> 6
- net /ROW1: track 271.4 -> 303.6 mm, vias 0 -> 3
- net Net-(LED31-DOUT): track 20.9 -> 23.6 mm, vias 0 -> 2
- net /COL8: track 76.3 -> 78.0 mm
- net Net-(LED29-DOUT): track 25.6 -> 24.2 mm
- net GND: track 0.26 -> 1.49 mm
- net Net-(LED30-DIN): track 20.7 -> 21.4 mm, vias 0 -> 2
- net /COL5: vias 6 -> 8
